File: PCB/ST32_SDR/PowerSupplay.sch (KiCad schematic (older format))
At the start: 1 part, among them U12 STM32F103C8Tx

Commit message: MCU schematics updated LCD Interface
Parts:
- removed U12: STM32F103C8Tx, Housings_QFP:LQFP-48_7x7mm_Pitch0.5mm, symbol STM32F103C8Tx
Changed lines of the file:
@@
 $Descr A4 11693 8268
 encoding utf-8
-Sheet 2 6
+Sheet 1 6
 Title ""
 Date ""
@@
 Comment4 ""
 $EndDescr
-$Comp
-L STM32F103C8Tx U12
-U 1 1 5DC33740
-P 5650 3350
-F 0 "U12" H 2850 5075 50  0000 L BNN
-F 1 "STM32F103C8Tx" H 8450 5075 50  0000 R BNN
-F 2 "Housings_QFP:LQFP-48_7x7mm_Pitch0.5mm" H 8450 5025 50  0001 R TNN
-F 3 "" H 5650 3350 50  0001 C CNN
-	1    5650 3350
-	1    0    0    -1
-$EndComp
 $EndSCHEMATC
