File: PCB/ST32_SDR/PowerSupplay.sch (KiCad schematic (older format))
At the start: 24 parts, among them U21 AP1117-33, U22 78M09, U23 MC34063, U24 MC34063

Commit message: update schematics
Parts:
- added C25: 330uF, symbol CP_Small
- added C26: 100nF, symbol C_Small
- added L1: 280uH, symbol L_Small
Connections:
- net +3V3: now also C25.1, C26.1, L1.1, L1.2
- net GND: now also C25.2, C26.2
Changed lines of the file:
@@
 LIBS:contrib
 LIBS:LCSDR
-LIBS:Logic_74xx
-LIBS:Logic_CMOS_4000
 LIBS:4ms-ic
-LIBS:Connector
 LIBS:Display
 LIBS:TRXklopik
+LIBS:stm32
+LIBS:switches
+LIBS:cmos4000
+LIBS:conn
 LIBS:LCSDR-cache
 EELAYER 25 0
@@
 $EndComp
 $Comp
-L GND #PWR203
+L GND #PWR079
 U 1 1 5DD9A087
 P 4600 1900
-F 0 "#PWR203" H 4600 1650 50  0001 C CNN
+F 0 "#PWR079" H 4600 1650 50  0001 C CNN
 F 1 "GND" H 4600 1750 50  0001 C CNN
 F 2 "" H 4600 1900 50  0001 C CNN
@@
 Connection ~ 3950 2400
 $Comp
-L GND #PWR197
+L GND #PWR080
 U 1 1 5DD9A371
 P 3600 2250
-F 0 "#PWR197" H 3600 2000 50  0001 C CNN
+F 0 "#PWR080" H 3600 2000 50  0001 C CNN
 F 1 "GND" H 3600 2100 50  0001 C CNN
 F 2 "" H 3600 2250 50  0001 C CNN
@@
 $EndComp
 $Comp
-L GND #PWR195
+L GND #PWR081
 U 1 1 5DD9A42B
 P 3400 2150
-F 0 "#PWR195" H 3400 1900 50  0001 C CNN
+F 0 "#PWR081" H 3400 1900 50  0001 C CNN
 F 1 "GND" H 3400 2000 50  0001 C CNN
 F 2 "" H 3400 2150 50  0001 C CNN
@@
 Connection ~ 2150 1350
 $Comp
-L +12V #PWR180
+L +12V #PWR082
 U 1 1 5DD9A4E4
 P 1250 2000
-F 0 "#PWR180" H 1250 1850 50  0001 C CNN
+F 0 "#PWR082" H 1250 1850 50  0001 C CNN
 F 1 "+12V" V 1250 2250 50  0000 C CNN
 F 2 "" H 1250 2000 50  0001 C CNN
@@
 $EndComp
 $Comp
-L +12V #PWR187
+L +12V #PWR083
 U 1 1 5DD9C169
 P 2300 3050
-F 0 "#PWR187" H 2300 2900 50  0001 C CNN
+F 0 "#PWR083" H 2300 2900 50  0001 C CNN
 F 1 "+12V" V 2300 3300 50  0000 C CNN
 F 2 "" H 2300 3050 50  0001 C CNN
@@
 $EndComp
 $Comp
-L +9V #PWR201
+L +9V #PWR084
 U 1 1 5DD9C2C5
 P 4400 2400
-F 0 "#PWR201" H 4400 2250 50  0001 C CNN
+F 0 "#PWR084" H 4400 2250 50  0001 C CNN
 F 1 "+9V" V 4400 2600 50  0000 C CNN
 F 2 "" H 4400 2400 50  0001 C CNN
@@
 $EndComp
 $Comp
-L +9V #PWR191
+L +9V #PWR085
 U 1 1 5DD9C3E9
 P 2900 3050
-F 0 "#PWR191" H 2900 2900 50  0001 C CNN
+F 0 "#PWR085" H 2900 2900 50  0001 C CNN
 F 1 "+9V" V 2900 3250 50  0000 C CNN
 F 2 "" H 2900 3050 50  0001 C CNN
@@
 $EndComp
 $Comp
-L GND #PWR189
+L GND #PWR086
 U 1 1 5DD9C454
 P 2600 3350
-F 0 "#PWR189" H 2600 3100 50  0001 C CNN
+F 0 "#PWR086" H 2600 3100 50  0001 C CNN
 F 1 "GND" H 2600 3200 50  0001 C CNN
 F 2 "" H 2600 3350 50  0001 C CNN
@@
 $EndComp
 $Comp
-L GND #PWR193
+L GND #PWR087
 U 1 1 5DD9C4CE
 P 3250 2650
-F 0 "#PWR193" H 3250 2400 50  0001 C CNN
+F 0 "#PWR087" H 3250 2400 50  0001 C CNN
 F 1 "GND" H 3250 2500 50  0001 C CNN
 F 2 "" H 3250 2650 50  0001 C CNN
@@
 $EndComp
 $Comp
-L GND #PWR199
+L GND #PWR088
 U 1 1 5DD9C50C
 P 3950 2650
-F 0 "#PWR199" H 3950 2400 50  0001 C CNN
+F 0 "#PWR088" H 3950 2400 50  0001 C CNN
 F 1 "GND" H 3950 2500 50  0001 C CNN
 F 2 "" H 3950 2650 50  0001 C CNN
@@
 $EndComp
 $Comp
-L GND #PWR185
+L GND #PWR089
 U 1 1 5DD9C54A
 P 2100 2650
-F 0 "#PWR185" H 2100 2400 50  0001 C CNN
+F 0 "#PWR089" H 2100 2400 50  0001 C CNN
 F 1 "GND" H 2100 2500 50  0001 C CNN
 F 2 "" H 2100 2650 50  0001 C CNN
@@
 $EndComp
 $Comp
-L GND #PWR183
+L GND #PWR090
 U 1 1 5DD9C5AC
 P 1650 2300
-F 0 "#PWR183" H 1650 2050 50  0001 C CNN
+F 0 "#PWR090" H 1650 2050 50  0001 C CNN
 F 1 "GND" H 1650 2150 50  0001 C CNN
 F 2 "" H 1650 2300 50  0001 C CNN
@@
 $EndComp
 $Comp
-L GND #PWR202
+L GND #PWR091
 U 1 1 5DD9C919
 P 4550 4450
-F 0 "#PWR202" H 4550 4200 50  0001 C CNN
+F 0 "#PWR091" H 4550 4200 50  0001 C CNN
 F 1 "GND" H 4550 4300 50  0001 C CNN
 F 2 "" H 4550 4450 50  0001 C CNN
@@
 Connection ~ 3900 4950
 $Comp
-L GND #PWR196
+L GND #PWR092
 U 1 1 5DD9C936
 P 3550 4800
-F 0 "#PWR196" H 3550 4550 50  0001 C CNN
+F 0 "#PWR092" H 3550 4550 50  0001 C CNN
 F 1 "GND" H 3550 4650 50  0001 C CNN
 F 2 "" H 3550 4800 50  0001 C CNN
@@
 $EndComp
 $Comp
-L GND #PWR194
+L GND #PWR093
 U 1 1 5DD9C93C
 P 3350 4700
-F 0 "#PWR194" H 3350 4450 50  0001 C CNN
+F 0 "#PWR093" H 3350 4450 50  0001 C CNN
 F 1 "GND" H 3350 4550 50  0001 C CNN
 F 2 "" H 3350 4700 50  0001 C CNN
@@
 Connection ~ 4100 4950
 $Comp
-L +12V #PWR186
+L +12V #PWR094
 U 1 1 5DD9C967
 P 2250 5600
-F 0 "#PWR186" H 2250 5450 50  0001 C CNN
+F 0 "#PWR094" H 2250 5450 50  0001 C CNN
 F 1 "+12V" V 2250 5850 50  0000 C CNN
 F 2 "" H 2250 5600 50  0001 C CNN
@@
 $EndComp
 $Comp
-L GND #PWR188
+L GND #PWR095
 U 1 1 5DD9C97A
 P 2550 5900
-F 0 "#PWR188" H 2550 5650 50  0001 C CNN
+F 0 "#PWR095" H 2550 5650 50  0001 C CNN
 F 1 "GND" H 2550 5750 50  0001 C CNN
 F 2 "" H 2550 5900 50  0001 C CNN
@@
 $EndComp
 $Comp
-L GND #PWR192
+L GND #PWR096
 U 1 1 5DD9C980
 P 3200 5200
-F 0 "#PWR192" H 3200 4950 50  0001 C CNN
+F 0 "#PWR096" H 3200 4950 50  0001 C CNN
 F 1 "GND" H 3200 5050 50  0001 C CNN
 F 2 "" H 3200 5200 50  0001 C CNN
@@
 $EndComp
 $Comp
-L GND #PWR198
+L GND #PWR097
 U 1 1 5DD9C986
 P 3900 5200
-F 0 "#PWR198" H 3900 4950 50  0001 C CNN
+F 0 "#PWR097" H 3900 4950 50  0001 C CNN
 F 1 "GND" H 3900 5050 50  0001 C CNN
 F 2 "" H 3900 5200 50  0001 C CNN
@@
 $EndComp
 $Comp
-L GND #PWR184
+L GND #PWR098
 U 1 1 5DD9C98C
 P 2050 5200
-F 0 "#PWR184" H 2050 4950 50  0001 C CNN
+F 0 "#PWR098" H 2050 4950 50  0001 C CNN
 F 1 "GND" H 2050 5050 50  0001 C CNN
 F 2 "" H 2050 5200 50  0001 C CNN
@@
 $EndComp
 $Comp
-L GND #PWR182
+L GND #PWR099
 U 1 1 5DD9C992
 P 1600 4850
-F 0 "#PWR182" H 1600 4600 50  0001 C CNN
+F 0 "#PWR099" H 1600 4600 50  0001 C CNN
 F 1 "GND" H 1600 4700 50  0001 C CNN
 F 2 "" H 1600 4850 50  0001 C CNN
@@
 $EndComp
 $Comp
-L +9V #PWR181
+L +9V #PWR0100
 U 1 1 5DD9CCE8
 P 1400 4550
-F 0 "#PWR181" H 1400 4400 50  0001 C CNN
+F 0 "#PWR0100" H 1400 4400 50  0001 C CNN
 F 1 "+9V" V 1400 4750 50  0000 C CNN
 F 2 "" H 1400 4550 50  0001 C CNN
@@
 $EndComp
 $Comp
-L +3.3V #PWR200
+L +3.3V #PWR0101
 U 1 1 5DD9CE73
 P 4350 4950
-F 0 "#PWR200" H 4350 4800 50  0001 C CNN
+F 0 "#PWR0101" H 4350 4800 50  0001 C CNN
 F 1 "+3.3V" V 4350 5200 50  0000 C CNN
 F 2 "" H 4350 4950 50  0001 C CNN
@@
 $EndComp
 $Comp
-L +3.3V #PWR190
+L +3.3V #PWR0102
 U 1 1 5DD9D384
 P 2850 5600
-F 0 "#PWR190" H 2850 5450 50  0001 C CNN
+F 0 "#PWR0102" H 2850 5450 50  0001 C CNN
 F 1 "+3.3V" V 2850 5850 50  0000 C CNN
 F 2 "" H 2850 5600 50  0001 C CNN
@@
 	0    1    1    0
 $EndComp
+$Comp
+L L_Small L1
+U 1 1 5DDE4A61
+P 5950 4950
+F 0 "L1" V 6150 5000 50  0000 L CNN
+F 1 "280uH" V 6050 4850 50  0000 L CNN
+F 2 "" H 5950 4950 50  0001 C CNN
+F 3 "" H 5950 4950 50  0001 C CNN
+	1    5950 4950
+	0    -1   -1   0
+$EndComp
+$Comp
+L +3.3V #PWR0103
+U 1 1 5DDE4F01
+P 5700 4950
+F 0 "#PWR0103" H 5700 4800 50  0001 C CNN
+F 1 "+3.3V" V 5700 5200 50  0000 C CNN
+F 2 "" H 5700 4950 50  0001 C CNN
+F 3 "" H 5700 4950 50  0001 C CNN
+	1    5700 4950
+	0    -1   -1   0
+$EndComp
+Wire Wire Line
+	5700 4950 5850 4950
+$Comp
+L +3V3 #PWR0104
+U 1 1 5DDE50CB
+P 6800 4950
+F 0 "#PWR0104" H 6800 4800 50  0001 C CNN
+F 1 "+3V3" V 6800 5200 50  0000 C CNN
+F 2 "" H 6800 4950 50  0001 C CNN
+F 3 "" H 6800 4950 50  0001 C CNN
+	1    6800 4950
+	0    1    1    0
+$EndComp
+Wire Wire Line
+	6050 4950 6800 4950
+$Comp
+L CP_Small C25
+U 1 1 5DDE528C
+P 6200 5100
+F 0 "C25" H 6300 5150 50  0000 L CNN
+F 1 "330uF" H 6300 5050 50  0000 L CNN
+F 2 "" H 6200 5100 50  0001 C CNN
+F 3 "" H 6200 5100 50  0001 C CNN
+	1    6200 5100
+	1    0    0    -1
+$EndComp
+$Comp
+L C_Small C26
+U 1 1 5DDE5430
+P 6700 5100
+F 0 "C26" H 6800 5150 50  0000 L CNN
+F 1 "100nF" H 6800 5050 50  0000 L CNN
+F 2 "" H 6700 5100 50  0001 C CNN
+F 3 "" H 6700 5100 50  0001 C CNN
+	1    6700 5100
+	1    0    0    -1
+$EndComp
+$Comp
+L GND #PWR0105
+U 1 1 5DDE5565
+P 6200 5200
+F 0 "#PWR0105" H 6200 4950 50  0001 C CNN
+F 1 "GND" H 6200 5050 50  0001 C CNN
+F 2 "" H 6200 5200 50  0001 C CNN
+F 3 "" H 6200 5200 50  0001 C CNN
+	1    6200 5200
+	1    0    0    -1
+$EndComp
+$Comp
+L GND #PWR0106
+U 1 1 5DDE5612
+P 6700 5200
+F 0 "#PWR0106" H 6700 4950 50  0001 C CNN
+F 1 "GND" H 6700 5050 50  0001 C CNN
+F 2 "" H 6700 5200 50  0001 C CNN
+F 3 "" H 6700 5200 50  0001 C CNN
+	1    6700 5200
+	1    0    0    -1
+$EndComp
+Wire Wire Line
+	6200 5000 6200 4950
+Connection ~ 6200 4950
+Wire Wire Line
+	6700 5000 6700 4950
+Connection ~ 6700 4950
 $EndSCHEMATC

Commit message: begin PCB
Parts:
- removed C121, C122: CP_Small, symbol CP_Small
- removed C123, C124, C127, C128: 1000uF, symbol CP_Small
- removed C125: 200pF, symbol C_Small
- removed C126: 360pF, symbol C_Small
- removed L29: 19uH, symbol L_Small
- removed L30: 15uH, symbol L_Small
- removed R86, R87, R88, R89: 0.49R, symbol R_Small
- removed R90: 11k, symbol R_Small
- removed R91: 1k, symbol R_Small
- removed R92: 18k, symbol R_Small
- removed R93: 6.2k, symbol R_Small
- removed U21: AP1117-33, TO_SOT_Packages_SMD:SOT-223-3_TabPin2, symbol AP1117-33
- removed U22: 78M09, symbol L7809
- removed U23, U24: MC34063, symbol MC34063
- added C36, C37: 10uF, Capacitors_ThroughHole:CP_Radial_D4.0mm_P2.00mm, symbol CP_Small
- added C38, C39, C42, C43: 1000uF, Capacitors_ThroughHole:CP_Radial_D10.0mm_P5.00mm, symbol CP_Small
- added C40: 200pF, UI:C_1206_0603, symbol C_Small
- added C41: 360pF, UI:C_1206_0603, symbol C_Small
- added J5: USB_B_Mini, Connect:USB_Mini-B, symbol USB_B_Mini
- added L2: 19uH, Choke_Axial_ThroughHole:Choke_Horizontal_RM10mm, symbol L_Small
- added L3: 15uH, Choke_Axial_ThroughHole:Choke_Horizontal_RM10mm, symbol L_Small
- added R10, R11, R12, R9: 0.49R, Resistors_ThroughHole:R_Axial_DIN0207_L6.3mm_D2.5mm_P10.16mm_Horizontal, symbol R_Small
- added R13: 11k, UI:R_1206_0603, symbol R_Small
- added R14: 1k, UI:R_1206_0603, symbol R_Small
- added R15: 18k, UI:R_1206_0603, symbol R_Small
- added R16: 6.2k, UI:R_1206_0603, symbol R_Small
- added R17, R18: 33, UI:R_1206_0603, symbol R_Small
- added U4: AP1117-33, TO_SOT_Packages_SMD:SOT-223, symbol AP1117-33
- added U5, U6: MC34063, UI:SOIC-8_3.9x4.9mm_Pitch1.27mm, symbol MC34063
- added U7: 78M09, TO_SOT_Packages_SMD:TO-252-2_Rectifier, symbol L7809
- C25: footprint (none) -> Capacitors_ThroughHole:CP_Radial_D10.0mm_P5.00mm
- C26: footprint (none) -> UI:C_1206_0603
- D2, D3: footprint (none) -> Diodes_SMD:D_SMA_Handsoldering
- L1: footprint (none) -> Choke_Axial_ThroughHole:Choke_Horizontal_RM10mm
Connections:
- net +12V: now also C37.1, R10.1, R12.2, U4.3 (VI), U6.6 (Vcc), U7.1 (IN)
- net +3V3: now also C38.1, C42.1, L2.2, R15.1, U4.2 (VO)
- net +9V: now also C36.1, C39.1, C43.1, L3.2, R11.2, R16.1, R9.1, U5.6 (Vcc), U7.3 (OUT)
- net GND: now also C36.2, C37.2, C38.2, C39.2, C40.2, C41.2, C42.2, C43.2, J5.5 (GND), J5.6 (Shield), R13.2, R14.2, U4.1 (GND), U5.4 (GND), U6.4 (GND), U7.2 (GND)
- net at D3.1 (K): now also L3.1, U6.2 (SWE)
- net at D2.1 (K): now also L2.1, U5.2 (SWE)
- new net: R10.2, R12.1, U6.1 (SWC), U6.7 (Ipk), U6.8 (DRC)
- new net: C41.1, U6.3 (TC)
- new net: R14.1, R16.2, U6.5 (CII)
- new net: R11.1, R9.2, U5.1 (SWC), U5.7 (Ipk), U5.8 (DRC)
- new net: C40.1, U5.3 (TC)
- new net: R13.1, R15.2, U5.5 (CII)
- new net: J5.2 (D-), R18.1
- new net: J5.3 (D+), R17.1
- new net USB_DM: R18.2
- new net USB_DP: R17.2

Commit message: PCB update
Parts:
- L2, L3: footprint Choke_Axial_ThroughHole:Choke_Horizontal_RM10mm -> Choke_Toroid_ThroughHole:Choke_Toroid_5x10mm_Vertical
Connections:
- net +12V: no longer U4.3 (VI)
- net +9V: now also U4.3 (VI)
Changed lines of the file:
@@
 Connection ~ 2100 2400
 $Comp
-L GND #PWR079
+L GND #PWR075
 U 1 1 5DD9A087
 P 4600 1900
-F 0 "#PWR079" H 4600 1650 50  0001 C CNN
+F 0 "#PWR075" H 4600 1650 50  0001 C CNN
 F 1 "GND" H 4600 1750 50  0001 C CNN
 F 2 "" H 4600 1900 50  0001 C CNN
@@
 Connection ~ 3950 2400
 $Comp
-L GND #PWR080
+L GND #PWR076
 U 1 1 5DD9A371
 P 3600 2250
-F 0 "#PWR080" H 3600 2000 50  0001 C CNN
+F 0 "#PWR076" H 3600 2000 50  0001 C CNN
 F 1 "GND" H 3600 2100 50  0001 C CNN
 F 2 "" H 3600 2250 50  0001 C CNN
@@
 $EndComp
 $Comp
-L GND #PWR081
+L GND #PWR077
 U 1 1 5DD9A42B
 P 3400 2150
-F 0 "#PWR081" H 3400 1900 50  0001 C CNN
+F 0 "#PWR077" H 3400 1900 50  0001 C CNN
 F 1 "GND" H 3400 2000 50  0001 C CNN
 F 2 "" H 3400 2150 50  0001 C CNN
@@
 Connection ~ 2150 1350
 $Comp
-L +12V #PWR082
+L +12V #PWR078
 U 1 1 5DD9A4E4
 P 1250 2000
-F 0 "#PWR082" H 1250 1850 50  0001 C CNN
+F 0 "#PWR078" H 1250 1850 50  0001 C CNN
 F 1 "+12V" V 1250 2250 50  0000 C CNN
 F 2 "" H 1250 2000 50  0001 C CNN
@@
 Connection ~ 4150 2400
 $Comp
-L +12V #PWR083
+L +12V #PWR079
 U 1 1 5DD9C169
 P 2700 3250
-F 0 "#PWR083" H 2700 3100 50  0001 C CNN
+F 0 "#PWR079" H 2700 3100 50  0001 C CNN
 F 1 "+12V" V 2700 3500 50  0000 C CNN
 F 2 "" H 2700 3250 50  0001 C CNN
@@
 $EndComp
 $Comp
-L +9V #PWR084
+L +9V #PWR080
 U 1 1 5DD9C2C5
 P 4400 2400
-F 0 "#PWR084" H 4400 2250 50  0001 C CNN
+F 0 "#PWR080" H 4400 2250 50  0001 C CNN
 F 1 "+9V" V 4400 2600 50  0000 C CNN
 F 2 "" H 4400 2400 50  0001 C CNN
@@
 $EndComp
 $Comp
-L +9V #PWR085
+L +9V #PWR081
 U 1 1 5DD9C3E9
 P 3300 3250
-F 0 "#PWR085" H 3300 3100 50  0001 C CNN
+F 0 "#PWR081" H 3300 3100 50  0001 C CNN
 F 1 "+9V" V 3300 3450 50  0000 C CNN
 F 2 "" H 3300 3250 50  0001 C CNN
@@
 $EndComp
 $Comp
-L GND #PWR086
+L GND #PWR082
 U 1 1 5DD9C454
 P 3000 3550
-F 0 "#PWR086" H 3000 3300 50  0001 C CNN
+F 0 "#PWR082" H 3000 3300 50  0001 C CNN
 F 1 "GND" H 3000 3400 50  0001 C CNN
 F 2 "" H 3000 3550 50  0001 C CNN
@@
 $EndComp
 $Comp
-L GND #PWR087
+L GND #PWR083
 U 1 1 5DD9C4CE
 P 3250 2650
-F 0 "#PWR087" H 3250 2400 50  0001 C CNN
+F 0 "#PWR083" H 3250 2400 50  0001 C CNN
 F 1 "GND" H 3250 2500 50  0001 C CNN
 F 2 "" H 3250 2650 50  0001 C CNN
@@
 $EndComp
 $Comp
-L GND #PWR088
+L GND #PWR084
 U 1 1 5DD9C50C
 P 3950 2650
-F 0 "#PWR088" H 3950 2400 50  0001 C CNN
+F 0 "#PWR084" H 3950 2400 50  0001 C CNN
 F 1 "GND" H 3950 2500 50  0001 C CNN
 F 2 "" H 3950 2650 50  0001 C CNN
@@
 $EndComp
 $Comp
-L GND #PWR089
+L GND #PWR085
 U 1 1 5DD9C54A
 P 2100 2650
-F 0 "#PWR089" H 2100 2400 50  0001 C CNN
+F 0 "#PWR085" H 2100 2400 50  0001 C CNN
 F 1 "GND" H 2100 2500 50  0001 C CNN
 F 2 "" H 2100 2650 50  0001 C CNN
@@
 $EndComp
 $Comp
-L GND #PWR090
+L GND #PWR086
 U 1 1 5DD9C5AC
 P 1650 2300
-F 0 "#PWR090" H 1650 2050 50  0001 C CNN
+F 0 "#PWR086" H 1650 2050 50  0001 C CNN
 F 1 "GND" H 1650 2150 50  0001 C CNN
 F 2 "" H 1650 2300 50  0001 C CNN
@@
 Connection ~ 2050 4950
 $Comp
-L GND #PWR091
+L GND #PWR087
 U 1 1 5DD9C919
 P 4550 4450
-F 0 "#PWR091" H 4550 4200 50  0001 C CNN
+F 0 "#PWR087" H 4550 4200 50  0001 C CNN
 F 1 "GND" H 4550 4300 50  0001 C CNN
 F 2 "" H 4550 4450 50  0001 C CNN
@@
 Connection ~ 3900 4950
 $Comp
-L GND #PWR092
+L GND #PWR088
 U 1 1 5DD9C936
 P 3550 4800
-F 0 "#PWR092" H 3550 4550 50  0001 C CNN
+F 0 "#PWR088" H 3550 4550 50  0001 C CNN
 F 1 "GND" H 3550 4650 50  0001 C CNN
 F 2 "" H 3550 4800 50  0001 C CNN
@@
 $EndComp
 $Comp
-L GND #PWR093
+L GND #PWR089
 U 1 1 5DD9C93C
 P 3350 4700
-F 0 "#PWR093" H 3350 4450 50  0001 C CNN
+F 0 "#PWR089" H 3350 4450 50  0001 C CNN
 F 1 "GND" H 3350 4550 50  0001 C CNN
 F 2 "" H 3350 4700 50  0001 C CNN
@@
 Connection ~ 4100 4950
 $Comp
-L +12V #PWR094
-U 1 1 5DD9C967
-P 2250 5600
-F 0 "#PWR094" H 2250 5450 50  0001 C CNN
-F 1 "+12V" V 2250 5850 50  0000 C CNN
-F 2 "" H 2250 5600 50  0001 C CNN
-F 3 "" H 2250 5600 50  0001 C CNN
-	1    2250 5600
-	0    -1   -1   0
-$EndComp
-$Comp
-L GND #PWR095
+L GND #PWR091
 U 1 1 5DD9C97A
 P 2550 5900
-F 0 "#PWR095" H 2550 5650 50  0001 C CNN
+F 0 "#PWR091" H 2550 5650 50  0001 C CNN
 F 1 "GND" H 2550 5750 50  0001 C CNN
 F 2 "" H 2550 5900 50  0001 C CNN
@@
 $EndComp
 $Comp
-L GND #PWR096
+L GND #PWR092
 U 1 1 5DD9C980
 P 3200 5200
-F 0 "#PWR096" H 3200 4950 50  0001 C CNN
+F 0 "#PWR092" H 3200 4950 50  0001 C CNN
 F 1 "GND" H 3200 5050 50  0001 C CNN
 F 2 "" H 3200 5200 50  0001 C CNN
@@
 $EndComp
 $Comp
-L GND #PWR097
+L GND #PWR093
 U 1 1 5DD9C986
 P 3900 5200
-F 0 "#PWR097" H 3900 4950 50  0001 C CNN
+F 0 "#PWR093" H 3900 4950 50  0001 C CNN
 F 1 "GND" H 3900 5050 50  0001 C CNN
 F 2 "" H 3900 5200 50  0001 C CNN
@@
 $EndComp
 $Comp
-L GND #PWR098
+L GND #PWR094
 U 1 1 5DD9C98C
 P 2050 5200
-F 0 "#PWR098" H 2050 4950 50  0001 C CNN
+F 0 "#PWR094" H 2050 4950 50  0001 C CNN
 F 1 "GND" H 2050 5050 50  0001 C CNN
 F 2 "" H 2050 5200 50  0001 C CNN
@@
 $EndComp
 $Comp
-L GND #PWR099
+L GND #PWR095
 U 1 1 5DD9C992
 P 1600 4850
-F 0 "#PWR099" H 1600 4600 50  0001 C CNN
+F 0 "#PWR095" H 1600 4600 50  0001 C CNN
 F 1 "GND" H 1600 4700 50  0001 C CNN
 F 2 "" H 1600 4850 50  0001 C CNN
@@
 $EndComp
 $Comp
-L +9V #PWR0100
+L +9V #PWR096
 U 1 1 5DD9CCE8
 P 1400 4550
-F 0 "#PWR0100" H 1400 4400 50  0001 C CNN
+F 0 "#PWR096" H 1400 4400 50  0001 C CNN
 F 1 "+9V" V 1400 4750 50  0000 C CNN
 F 2 "" H 1400 4550 50  0001 C CNN
@@
 $EndComp
 $Comp
-L +3.3V #PWR0101
+L +3.3V #PWR097
 U 1 1 5DD9CE73
 P 4350 4950
-F 0 "#PWR0101" H 4350 4800 50  0001 C CNN
+F 0 "#PWR097" H 4350 4800 50  0001 C CNN
 F 1 "+3.3V" V 4350 5200 50  0000 C CNN
 F 2 "" H 4350 4950 50  0001 C CNN
@@
 $EndComp
 $Comp
-L +3.3V #PWR0102
+L +3.3V #PWR098
 U 1 1 5DD9D384
 P 2850 5600
-F 0 "#PWR0102" H 2850 5450 50  0001 C CNN
+F 0 "#PWR098" H 2850 5450 50  0001 C CNN
 F 1 "+3.3V" V 2850 5850 50  0000 C CNN
 F 2 "" H 2850 5600 50  0001 C CNN
@@
 $EndComp
 $Comp
-L +3.3V #PWR0103
+L +3.3V #PWR099
 U 1 1 5DDE4F01
 P 5700 4950
-F 0 "#PWR0103" H 5700 4800 50  0001 C CNN
+F 0 "#PWR099" H 5700 4800 50  0001 C CNN
 F 1 "+3.3V" V 5700 5200 50  0000 C CNN
 F 2 "" H 5700 4950 50  0001 C CNN
@@
 	5700 4950 5850 4950
 $Comp
-L +3V3 #PWR0104
+L +3V3 #PWR0100
 U 1 1 5DDE50CB
 P 6800 4950
-F 0 "#PWR0104" H 6800 4800 50  0001 C CNN
+F 0 "#PWR0100" H 6800 4800 50  0001 C CNN
 F 1 "+3V3" V 6800 5200 50  0000 C CNN
 F 2 "" H 6800 4950 50  0001 C CNN
@@
 $EndComp
 $Comp
-L GND #PWR0105
+L GND #PWR0101
 U 1 1 5DDE5565
 P 6200 5200
-F 0 "#PWR0105" H 6200 4950 50  0001 C CNN
+F 0 "#PWR0101" H 6200 4950 50  0001 C CNN
 F 1 "GND" H 6200 5050 50  0001 C CNN
 F 2 "" H 6200 5200 50  0001 C CNN
@@
 $EndComp
 $Comp
-L GND #PWR0106
+L GND #PWR0102
 U 1 1 5DDE5612
 P 6700 5200
-F 0 "#PWR0106" H 6700 4950 50  0001 C CNN
+F 0 "#PWR0102" H 6700 4950 50  0001 C CNN
 F 1 "GND" H 6700 5050 50  0001 C CNN
 F 2 "" H 6700 5200 50  0001 C CNN
@@
 F 0 "L3" H 4200 2200 50  0000 L CNN
 F 1 "15uH" H 4200 2100 50  0000 L CNN
-F 2 "Choke_Axial_ThroughHole:Choke_Horizontal_RM10mm" H 4150 2150 50  0001 C CNN
+F 2 "Choke_Toroid_ThroughHole:Choke_Toroid_5x10mm_Vertical" H 4150 2150 50  0001 C CNN
 F 3 "" H 4150 2150 50  0001 C CNN
 	1    4150 2150
@@
 F 0 "L2" H 4150 4750 50  0000 L CNN
 F 1 "19uH" H 4150 4650 50  0000 L CNN
-F 2 "Choke_Axial_ThroughHole:Choke_Horizontal_RM10mm" H 4100 4700 50  0001 C CNN
+F 2 "Choke_Toroid_ThroughHole:Choke_Toroid_5x10mm_Vertical" H 4100 4700 50  0001 C CNN
 F 3 "" H 4100 4700 50  0001 C CNN
 	1    4100 4700
@@
 USB_DP
 $Comp
-L GND #PWR0107
+L GND #PWR0103
 U 1 1 5DDFC12C
 P 8500 2350
-F 0 "#PWR0107" H 8500 2100 50  0001 C CNN
+F 0 "#PWR0103" H 8500 2100 50  0001 C CNN
 F 1 "GND" H 8500 2200 50  0000 C CNN
 F 2 "" H 8500 2350 50  0001 C CNN
@@
 	8500 2250 8500 2350
 Connection ~ 8500 2300
+$Comp
+L +9V #PWR?
+U 1 1 5DE21DEE
+P 2250 5600
+F 0 "#PWR?" H 2250 5450 50  0001 C CNN
+F 1 "+9V" V 2250 5800 50  0000 C CNN
+F 2 "" H 2250 5600 50  0001 C CNN
+F 3 "" H 2250 5600 50  0001 C CNN
+	1    2250 5600
+	0    -1   -1   0
+$EndComp
 $EndSCHEMATC
