File: PCB/ST32_SDR/LCSDR.sch (KiCad schematic (older format))
At the start: 238 parts, among them J2 LINE OUT, K1 LU-12, P1 BNC, P10 CONN_01X01, P11 CONN_01X01, P12 CONN_01X01, P13 CONN_01X01, P2 SPI, P4 PA_TX, P5 ENCODER, Q1 IRF510N, Q2 MMBT2222LT1G, Q3 BFG135, Q4 PMBT2907, Q5 PMBT2222, Q6 PMBT2222, T1 1:4, T2 1_9, U1 MC33179DR2G, U10 74LVC1G3157, U11 SN74LVC1G00DCKR, U14 74HC4053, U18 Si570, U2 PE4259ds, U25 PE4259ds, U26 PE4259ds, U27 LM78L06ACZ, U3 74LVC1G3157, U4 4053, U5 LD1117v25, U6 74HC4053, U7 SN74LVC1G00DCKR, U8 MC33179DR2G, U9 74LCX574, Y5 8Mhz

Commit message: recover LCD interface at MCU
Changed lines of the file:
@@
 	24250 8700 24250 8350
 Wire Wire Line
-	21000 8350 24250 8350
-Wire Wire Line
-	21000 4550 21000 8350
+	24250 8350 21000 8350
+Wire Wire Line
+	21000 8350 21000 4550
 Wire Wire Line
 	24950 9900 24950 9800
@@
 	20050 6900 20100 6900
 Wire Wire Line
-	20100 7150 20100 6900
-Wire Wire Line
-	14500 7150 20100 7150
+	20100 6900 20100 7150
+Wire Wire Line
+	20100 7150 14500 7150
 Wire Wire Line
 	15050 7150 15050 6900
@@
 	20050 7800 20100 7800
 Wire Wire Line
-	20100 8100 20100 7800
-Wire Wire Line
-	14800 8100 20100 8100
+	20100 7800 20100 8100
+Wire Wire Line
+	20100 8100 14800 8100
 Wire Wire Line
 	15050 8100 15050 7800
@@
 	9250 3500 9250 7150
 Wire Wire Line
-	8950 7150 9250 7150
+	9250 7150 8950 7150
 Wire Wire Line
 	6100 7400 6100 9350
