File: PCB/ST32_SDR/LCSDR.sch (KiCad schematic (older format))
At the start: 250 parts, among them CON1 +13,8v, J2 LINE OUT, K1 LU-12, P1 BNC, P10 CONN_01X01, P11 CONN_01X01, P12 CONN_01X01, P13 CONN_01X01, P2 SPI, P3 USB_OTG, P4 PA_TX, P5 ENCODER, Q1 IRF510N, Q2 MMBT2222LT1G, Q3 BFG135, Q4 PMBT2907, Q5 PMBT2222, Q6 PMBT2222, T1 1:4, T2 1_9, U1 MC33179DR2G, U10 74LVC1G3157, U11 SN74LVC1G00DCKR, U14 74HC4053, U15 L78M09, U18 Si570, U2 PE4259ds, U25 PE4259ds, U26 PE4259ds, U27 LM78L06ACZ, U3 74LVC1G3157, U4 4053, U5 LD1117v25, U6 74HC4053, U7 SN74LVC1G00DCKR, U8 MC33179DR2G, U9 74LCX574, Y5 8Mhz

Commit message: Schematics update
Parts:
- removed C74, C76, C78: 100nF, LCSDR:C_1206_0603, symbol C_Small
- removed C75: 330uF, LCSDR:C_Radial_D10_L13_P5, symbol CP1_Small
- removed C77: 100uF, LCSDR:C_Radial_D5_L11_P2.5, symbol CP1_Small
- removed C79: 10uF, LCSDR:Universal_C_Radial_D5_L11_P2_tantal, symbol CP1_Small
- removed CON1: +13,8v, LCSDR:BARREL_JACK, symbol BARREL_JACK-RESCUE-LCSDR
- removed D12: WE-TVS824011, TO_SOT_Packages_SMD:SOT-23-5_HandSoldering, symbol WE-TVS824011
- removed P3: USB_OTG, Connect:USB_Mini-B, symbol USB_OTG
- removed U15: L78M09, TO_SOT_Packages_SMD:TO-252-2_Rectifier, symbol LM7806ACT-RESCUE-LCSDR
Connections:
- wire segments 691 -> 898

Commit message: MCU schematics updated LCD Interface
Parts:
- removed C94: 100nF, LCSDR:C_1206_0603, symbol C_Small
- removed C95: 10uF, LCSDR:Universal_C_Radial_D5_L11_P2_tantal, symbol CP1_Small
Connections:
- wire segments 898 -> 639

Commit message: add LCD resistors
Parts:
- added C94: 100nF, LCSDR:C_1206_0603, symbol C_Small
- added C95: 10uF, LCSDR:Universal_C_Radial_D5_L11_P2_tantal, symbol CP1_Small
Connections:
- wire segments 639 -> 664

Commit message: update schematics
Parts:
- removed C1, C17, C2, C4, C46, C95: 10uF, LCSDR:Universal_C_Radial_D5_L11_P2_tantal, symbol CP1_Small
- removed C10, C100, C101, C102, C103, C21, C24, C25, C40, C54, C67, C81, C91: 1uF, LCSDR:C_1206_0603, symbol C_Small
- removed C104, C105, C106, C107, C108, C110, C111, C34, C56, C86, C93: 15nF, Capacitors_SMD:C_0603_HandSoldering, symbol C_Small
- removed C109: 15n, Capacitors_SMD:C_0603_HandSoldering, symbol C_Small
- removed C11, C12: 22pF, LCSDR:C_1206_0603, symbol C_Small
- removed C13, C52, C7, C8, C9: 10uF, Capacitors_Tantalum_SMD:CP_Tantalum_Case-A_EIA-3216-18_Hand, symbol CP1_Small
- removed C14, C15, C16, C18, C22, C29, C3, C31, C35, C47, C5, C53, C6, C68, C70, C72, C73, C82, C87, C89, C94, C96: 100nF, LCSDR:C_1206_0603, symbol C_Small
- removed C19, C30, C41, C48, C80: 10uF 16v, Capacitors_Tantalum_SMD:CP_Tantalum_Case-A_EIA-3216-18_Hand, symbol CP1_Small
- removed C20, C83, C92: 100uF, LCSDR:C_Radial_D5_L11_P2.5, symbol CP1_Small
- removed C23, C33, C43, C51: 27nF, LCSDR:C_1206_0603, symbol C_Small
- removed C26: 120pF, Capacitors_SMD:C_0603_HandSoldering, symbol C_Small
- removed C27, C28: 270pF, LCSDR:C_1206_0603, symbol C_Small
- removed C32, C36, C39: 680pF, Capacitors_SMD:C_0603_HandSoldering, symbol C_Small
- removed C37, C38, C45, C49: 820pF, Capacitors_SMD:C_0603_HandSoldering, symbol C_Small
- removed C42: 47uF, Capacitors_SMD:CP_Elec_6.3x7.7, symbol CP1_Small
- removed C44, C61, C65: 360pF, Capacitors_SMD:C_0603_HandSoldering, symbol C_Small
- removed C50, C62, C63: 33pF, Capacitors_SMD:C_0603_HandSoldering, symbol C_Small
- removed C55, C98: 1000uF, Capacitors_ThroughHole:CP_Radial_D8.0mm_P3.50mm, symbol CP1_Small
- removed C57, C97: 180pF, Capacitors_SMD:C_0603_HandSoldering, symbol C_Small
- removed C58, C66: 6.8uF, Capacitors_Tantalum_SMD:CP_Tantalum_Case-A_EIA-3216-18_Hand, symbol CP1_Small
- removed C59, C64: 10n, LCSDR:C_1206_0603, symbol C_Small
- removed C60, C69: 390p, Capacitors_SMD:C_0603_HandSoldering, symbol C_Small
- removed C71: 1n, LCSDR:C_1206_0603, symbol C_Small
- removed C84, C85, C88, C90: 4.7uF, Capacitors_SMD:C_0603_HandSoldering, symbol C_Small
- removed D1: LL4148, Diodes_SMD:D_MiniMELF_Handsoldering, symbol D
- removed D11: LED, LEDs:LED_D5.0mm, symbol LED-RESCUE-LCSDR
- removed J2: LINE OUT, LCSDR:audio_jack_3_5mm_PJ307, symbol JACK_TRS_3pins
- removed K1: LU-12, Relays_ThroughHole:Relay_SPDT_HJR-4102, symbol RELAY_1RT
- removed L1, L24, L26, L6: 100uH, LCSDR:Resistor_Horizontal_RM10mm, symbol L_Small
- removed L10, L22, L25, L3, L4, L5: 47uH, LCSDR:Resistor_Horizontal_RM10mm, symbol L_Small
- removed L11: 4.7uH, Resistors_SMD:R_1210_HandSoldering, symbol L_Small
- removed L12, L13: 472K, LCSDR:Resistor_Horizontal_RM10mm, symbol L_Small
- removed L14, L15, L16: 2.2uH, Resistors_SMD:R_1210_HandSoldering, symbol L_Small
- removed L17, L18, L19: 1uH, Resistors_SMD:R_1210_HandSoldering, symbol L_Small
- removed L2: 4.7uH, LCSDR:Choke_CD54, symbol L_Small
- removed L20, L21, L7: 470nH, Resistors_SMD:R_1210_HandSoldering, symbol L_Small
- removed L23: 0.47uH, Resistors_SMD:R_1210_HandSoldering, symbol L_Small
- removed L8, L9: 220nH, Resistors_SMD:R_1210_HandSoldering, symbol L_Small
- removed P1: BNC, LCSDR:BNC_Socket_TYCO-AMP, symbol BNC
- removed P10, P11, P12, P13: CONN_01X01, Mounting_Holes:MountingHole_3.2mm_M3_ISO7380_Pad, symbol CONN_01X01
- removed P2: SPI, Pin_Headers:Pin_Header_Straight_2x03_Pitch2.54mm, symbol CONN_02X03
- removed P4: PA_TX, Pin_Headers:Pin_Header_Straight_1x02_Pitch2.54mm, symbol CONN_01X02
- removed P5: ENCODER, Pin_Headers:Pin_Header_Straight_1x04_Pitch2.54mm, symbol CONN_01X04
- removed Q1: IRF510N, LCSDR:TO-220_Horizontal_Reversed, symbol IRF540N
- removed Q2: MMBT2222LT1G, TO_SOT_Packages_SMD:SOT-23_Handsoldering, symbol BC850
- removed Q3: BFG135, LCSDR:SOT-223, symbol BFG135
- removed Q4: PMBT2907, TO_SOT_Packages_SMD:SOT-23_Handsoldering, symbol Q_PNP_BEC
- removed Q5, Q6: PMBT2222, TO_SOT_Packages_SMD:SOT-23_Handsoldering, symbol BC850
- removed R1, R10, R18, R2, R21, R26, R27, R9: 3k 1%, Resistors_SMD:R_0603_HandSoldering, symbol R_Small
- removed R11, R12, R15, R16: 510R, LCSDR:R_1206_0603, symbol R_Small
- removed R13, R20: 47R, LCSDR:R_1206_0603, symbol R_Small
- removed R14, R50, R65: 10k, Resistors_SMD:R_0603_HandSoldering, symbol R_Small
- removed R17, R24, R33, R36: 20R, LCSDR:R_1206_0603, symbol R_Small
- removed R19, R28, R29, R30, R35, R6: 10k, LCSDR:R_1206_0603, symbol R_Small
- removed R22, R25, R3, R39, R45, R5: 1k 1%, Resistors_SMD:R_0603_HandSoldering, symbol R_Small
- removed R23, R4: 270R 1%, Resistors_SMD:R_0603_HandSoldering, symbol R_Small
- removed R31: 82R, LCSDR:R_1206_0603, symbol R_Small
- removed R32: 33R, Resistors_SMD:R_2512_HandSoldering, symbol R_Small
- removed R34, R58, R59: k91, LCSDR:R_1206_0603, symbol R_Small
- removed R37, R54: 13R, LCSDR:R_1206_0603, symbol R_Small
- removed R38: 20, Resistors_SMD:R_0603_HandSoldering, symbol R_Small
- removed R40, R42, R43, R46, R47: 4.7k 1%, Resistors_SMD:R_0603_HandSoldering, symbol R_Small
- removed R41: 51, Resistors_SMD:R_0603_HandSoldering, symbol R_Small
- removed R44, R49: 15, Resistors_SMD:R_0603_HandSoldering, symbol R_Small
- removed R48: 4k75, Resistors_SMD:R_0603_HandSoldering, symbol R_Small
- removed R52, R53: 82, Resistors_SMD:R_0603_HandSoldering, symbol R_Small
- removed R56: 33R, LCSDR:R_1206_0603, symbol R_Small
- removed R57: 5R1, LCSDR:R_1206_0603, symbol R_Small
- removed R60: k56, LCSDR:R_1206_0603, symbol R_Small
- removed R61, R64: 2.2k, Resistors_ThroughHole:R_Axial_DIN0204_L3.6mm_D1.6mm_P2.54mm_Vertical, symbol R_Small
- removed R62, R7, R70, R8: 1k, LCSDR:R_1206_0603, symbol R_Small
- removed R63: k510, LCSDR:R_1206_0603, symbol R_Small
- removed R66: 1k, Resistors_SMD:R_0603_HandSoldering, symbol R_Small
- removed R67: 1k5, LCSDR:R_1206_0603, symbol R_Small
- removed R68, R69: 2k2, LCSDR:R_1206_0603, symbol R_Small
- removed R71, R74: 1R, Resistors_SMD:R_0603_HandSoldering, symbol R_Small
- removed R72: 4.7k, LCSDR:R_1206_0603, symbol R_Small
- removed R73: 330, LCSDR:R_1206_0603, symbol R_Small
- removed RV1: 5k, Potentiometers:Potentiometer_Trimmer_Bourns_3296W, symbol POT-RESCUE-LCSDR
- removed T1: 1:4, LCSDR:TRANSF1_4, symbol 1:4
- removed T2: 1_9, LCSDR:HF1_9, symbol 1_9
- removed U1: MC33179DR2G, Housings_SOIC:SOIC-14_3.9x8.7mm_Pitch1.27mm, symbol MC33179DR2G-RESCUE-LCSDR
- removed U10, U3: 74LVC1G3157, TO_SOT_Packages_SMD:SOT-23-6_Handsoldering, symbol 74LVC1G3157
- removed U11, U7: SN74LVC1G00DCKR, TO_SOT_Packages_SMD:SOT-353_SC-70-5_Handsoldering, symbol NL17SV00
- removed U14, U6: 74HC4053, Housings_SOIC:SOIC-16_3.9x9.9mm_Pitch1.27mm, symbol 4053
- removed U18: Si570, Oscillators:Oscillator_SMD_SI570_SI571_HandSoldering, symbol Si570
- removed U2, U25, U26: PE4259ds, TO_SOT_Packages_SMD:SOT-363_SC-70-6_Handsoldering, symbol PE4259ds
- removed U27: LM78L06ACZ, TO_SOT_Packages_THT:TO-92_Inline_Wide, symbol LM78L05ACZ
- removed U4: 4053, symbol 4053
- removed U5: LD1117v25, LCSDR:SOT-223, symbol LD33
- removed U8: MC33179DR2G, LCSDR:SOIC-14_3.9x8.7mm_Pitch1.27mm, symbol MC33179DR2G-RESCUE-LCSDR
- removed U9: 74LCX574, Housings_SSOP:SSOP-20_5.3x7.2mm_Pitch0.65mm, symbol 74LCX574
- removed Y5: 8Mhz, Crystals:Crystal_HC49-U_Vertical, symbol Crystal
Connections:
- net labels removed: +13.8V, 0, 0_1, 0_2, 0_3, 180_1, 180_2, 180_3, 2,75V, 270_1, 270_2, 270_3, 90, 90_1, 90_2, 90_3, GND, MOSI
- wire segments 664 -> 0
Other:
- note removed: "10dB"
- note removed: "17..10M\n"
- note removed: "20M\n"
- note removed: "40M\n"
- note removed: "80M\n"

Commit message: UI PCB linux 1
Parts:
- added J10, J11, J8, J9: Conn_01x01, Mounting_Holes:MountingHole_3.2mm_M3_DIN965_Pad, symbol Conn_01x01
- added J6: IQ, Pin_Headers:Pin_Header_Straight_1x06_Pitch2.54mm, symbol Conn_01x06
- added J7: CLK, Pin_Headers:Pin_Header_Straight_1x06_Pitch2.54mm, symbol Conn_01x06
Connections:
- new net CLK0: J7.2 (Pin_2)
- new net CLK1: J7.4 (Pin_4)
- new net CLK2: J7.6 (Pin_6)
- new net GND: J10.1 (Pin_1), J11.1 (Pin_1), J7.1 (Pin_1), J7.3 (Pin_3), J7.5 (Pin_5), J8.1 (Pin_1), J9.1 (Pin_1)
- new net I_IN: J6.1 (Pin_1)
- new net Q_IN: J6.2 (Pin_2)
Changed lines of the file:
@@
 LIBS:4ms-ic
 LIBS:Display
-LIBS:switches
-LIBS:cmos4000
+LIBS:Connector
+LIBS:Relay
 LIBS:LCSDR-cache
 EELAYER 25 0
@@
 F1 "PowerSupplay.sch" 60
 $EndSheet
+$Comp
+L Conn_01x06 J6
+U 1 1 5DE239A8
+P 9700 1300
+F 0 "J6" H 9700 1600 50  0000 C CNN
+F 1 "IQ" H 9700 900 50  0000 C CNN
+F 2 "Pin_Headers:Pin_Header_Straight_1x06_Pitch2.54mm" H 9700 1300 50  0001 C CNN
+F 3 "" H 9700 1300 50  0001 C CNN
+	1    9700 1300
+	1    0    0    -1
+$EndComp
+Text GLabel 9050 1100 0    60   Output ~ 0
+I_IN
+Text GLabel 9050 1250 0    60   Output ~ 0
+Q_IN
+Wire Wire Line
+	9050 1100 9500 1100
+Wire Wire Line
+	9050 1250 9300 1250
+Wire Wire Line
+	9300 1250 9300 1200
+Wire Wire Line
+	9300 1200 9500 1200
+Text GLabel 9050 1400 0    60   Output ~ 0
+I2C_SCL
+Text GLabel 9050 1550 0    60   Output ~ 0
+I2C_SDA
+$Comp
+L Conn_01x06 J7
+U 1 1 5DE24552
+P 9700 2250
+F 0 "J7" H 9700 2550 50  0000 C CNN
+F 1 "CLK" H 9700 1850 50  0000 C CNN
+F 2 "Pin_Headers:Pin_Header_Straight_1x06_Pitch2.54mm" H 9700 2250 50  0001 C CNN
+F 3 "" H 9700 2250 50  0001 C CNN
+	1    9700 2250
+	1    0    0    -1
+$EndComp
+Text GLabel 9150 2150 0    60   Output ~ 0
+CLK0
+Text GLabel 9150 2350 0    60   Output ~ 0
+CLK1
+Text GLabel 9150 2550 0    60   Output ~ 0
+CLK2
+Wire Wire Line
+	9150 2150 9500 2150
+Wire Wire Line
+	9150 2350 9500 2350
+Wire Wire Line
+	9150 2550 9500 2550
+$Comp
+L GND #PWR01
+U 1 1 5DE248A0
+P 9450 2750
+F 0 "#PWR01" H 9450 2500 50  0001 C CNN
+F 1 "GND" H 9450 2600 50  0000 C CNN
+F 2 "" H 9450 2750 50  0001 C CNN
+F 3 "" H 9450 2750 50  0001 C CNN
+	1    9450 2750
+	1    0    0    -1
+$EndComp
+Wire Wire Line
+	9450 2050 9450 2750
+Wire Wire Line
+	9450 2450 9500 2450
+Wire Wire Line
+	9450 2250 9500 2250
+Connection ~ 9450 2450
+Wire Wire Line
+	9450 2050 9500 2050
+Connection ~ 9450 2250
+$Comp
+L Conn_01x01 J8
+U 1 1 5DE25479
+P 9450 5950
+F 0 "J8" H 9450 6050 50  0000 C CNN
+F 1 "Conn_01x01" H 9450 5850 50  0000 C CNN
+F 2 "Mounting_Holes:MountingHole_3.2mm_M3_DIN965_Pad" H 9450 5950 50  0001 C CNN
+F 3 "" H 9450 5950 50  0001 C CNN
+	1    9450 5950
+	0    -1   -1   0
+$EndComp
+$Comp
+L Conn_01x01 J9
+U 1 1 5DE254BB
+P 9800 5950
+F 0 "J9" H 9800 6050 50  0000 C CNN
+F 1 "Conn_01x01" H 9800 5850 50  0000 C CNN
+F 2 "Mounting_Holes:MountingHole_3.2mm_M3_DIN965_Pad" H 9800 5950 50  0001 C CNN
+F 3 "" H 9800 5950 50  0001 C CNN
+	1    9800 5950
+	0    -1   -1   0
+$EndComp
+$Comp
+L Conn_01x01 J10
+U 1 1 5DE254E5
+P 10150 5950
+F 0 "J10" H 10150 6050 50  0000 C CNN
+F 1 "Conn_01x01" H 10150 5850 50  0000 C CNN
+F 2 "Mounting_Holes:MountingHole_3.2mm_M3_DIN965_Pad" H 10150 5950 50  0001 C CNN
+F 3 "" H 10150 5950 50  0001 C CNN
+	1    10150 5950
+	0    -1   -1   0
+$EndComp
+$Comp
+L Conn_01x01 J11
+U 1 1 5DE2550E
+P 10500 5950
+F 0 "J11" H 10500 6050 50  0000 C CNN
+F 1 "Conn_01x01" H 10500 5850 50  0000 C CNN
+F 2 "Mounting_Holes:MountingHole_3.2mm_M3_DIN965_Pad" H 10500 5950 50  0001 C CNN
+F 3 "" H 10500 5950 50  0001 C CNN
+	1    10500 5950
+	0    -1   -1   0
+$EndComp
+$Comp
+L GND #PWR02
+U 1 1 5DE25560
+P 9450 6150
+F 0 "#PWR02" H 9450 5900 50  0001 C CNN
+F 1 "GND" H 9450 6000 50  0000 C CNN
+F 2 "" H 9450 6150 50  0001 C CNN
+F 3 "" H 9450 6150 50  0001 C CNN
+	1    9450 6150
+	1    0    0    -1
+$EndComp
+$Comp
+L GND #PWR03
+U 1 1 5DE25589
+P 9800 6150
+F 0 "#PWR03" H 9800 5900 50  0001 C CNN
+F 1 "GND" H 9800 6000 50  0000 C CNN
+F 2 "" H 9800 6150 50  0001 C CNN
+F 3 "" H 9800 6150 50  0001 C CNN
+	1    9800 6150
+	1    0    0    -1
+$EndComp
+$Comp
+L GND #PWR04
+U 1 1 5DE255A6
+P 10150 6150
+F 0 "#PWR04" H 10150 5900 50  0001 C CNN
+F 1 "GND" H 10150 6000 50  0000 C CNN
+F 2 "" H 10150 6150 50  0001 C CNN
+F 3 "" H 10150 6150 50  0001 C CNN
+	1    10150 6150
+	1    0    0    -1
+$EndComp
+$Comp
+L GND #PWR05
+U 1 1 5DE255C3
+P 10500 6150
+F 0 "#PWR05" H 10500 5900 50  0001 C CNN
+F 1 "GND" H 10500 6000 50  0000 C CNN
+F 2 "" H 10500 6150 50  0001 C CNN
+F 3 "" H 10500 6150 50  0001 C CNN
+	1    10500 6150
+	1    0    0    -1
+$EndComp
 $EndSCHEMATC
