File: PCB/ST32_SDR/MCU.sch (KiCad schematic (older format))
At the start: 13 parts, among them U17 FM24CL16B, U19 STM32F401RCTx, Y1 20Mhz

Commit message: begin PCB
Parts:
- removed C117, C119: C_Small, symbol C_Small
- removed C118, C120, C129, C130, C131, C132: 100nF, symbol C_Small
- removed R84, R85: 0*, symbol R_Small
- removed U17: FM24CL16B, Housings_SOIC:SOIC-8_3.9x4.9mm_Pitch1.27mm, symbol 24LC16
- removed U19: STM32F401RCTx, LQFP64, symbol STM32F401RCTx
- added C27, C29, C32, C33, C34, C35: 100nF, UI:C_1206_0603, symbol C_Small
- added C28, C30: 22, UI:C_1206_0603, symbol C_Small
- added R7, R8: 0*, UI:R_1206_0603, symbol R_Small
- added U2: FM24CL16B, Housings_SOIC:SOIC-8_3.9x4.9mm_Pitch1.27mm, symbol 24LC16
- added U3: STM32F401RCTx, Housings_QFP:LQFP-64_10x10mm_Pitch0.5mm, symbol STM32F401RCTx
- Y1: footprint (none) -> Crystals:Crystal_HC49-U_Vertical
Connections:
- net +3V3: now also C27.1, C33.2, C34.2, C35.2, U2.8 (VCC), U3.19 (VDD), U3.32 (VDD), U3.48 (VDD), U3.64 (VDD)
- net BAND0: now also U3.26 (ADC1_IN8/TIM1_CH2N/TIM3_CH3/PB0)
- net BAND1: now also U3.27 (ADC1_IN9/TIM1_CH3N/TIM3_CH4/PB1)
- net BAND2: now also U3.28 (BOOT1/PB2)
- net BAND3: now also U3.29 (I2C2_SCL/I2S2_CK/SPI2_SCK/TIM2_CH3/PB10)
- net ENCODER_A: now also U3.14 (ADC1_IN0/SYS_WKUP/TIM2_CH1/TIM2_ETR/TIM5_CH1/USART2_CTS/PA0)
- net ENCODER_B: now also U3.15 (ADC1_IN1/TIM2_CH2/TIM5_CH2/USART2_RTS/PA1)
- net GND: now also C27.2, C28.2, C29.2, C30.2, C32.2, C33.1, C34.1, C35.1, R7.1, R8.2, U2.4 (GND), U2.7 (WP), U3.12 (VSSA), U3.18 (VSS), U3.60 (BOOT0), U3.63 (VSS)
- net I2C_SCL: now also U2.6 (SCL), U3.61 (I2C1_SCL/SDIO_D4/TIM10_CH1/TIM4_CH3/PB8)
- net I2C_SDA: now also U2.5 (SDA), U3.62 (I2C1_SDA/I2S2_WS/SDIO_D5/SPI2_NSS/TIM11_CH1/TIM4_CH4/PB9)
- net I2S_LRCK: now also U3.33 (I2C2_SMBA/I2S2_WS/SPI2_NSS/TIM1_BKIN/PB12)
- net I2S_MCLK: now also U3.37 (PC6/I2S2_MCK/SDIO_D6/TIM3_CH1/USART6_TX)
- net I2S_SCLK: now also U3.34 (I2S2_CK/SPI2_SCK/TIM1_CH1N/PB13)
- net I2S_SDI: now also U3.35 (I2S2_ext_SD/SPI2_MISO/TIM1_CH2N/PB14)
- net I2S_SDO: now also U3.36 (ADC1_EXTI15/I2S2_SD/RTC_REFIN/SPI2_MOSI/TIM1_CH3N/PB15)
- net I_IN_M1: now also U3.56 (I2C3_SDA/I2S3_ext_SD/SPI1_MISO/SPI3_MISO/SYS_JTRST/TIM3_CH1/PB4)
- net I_IN_M2: now also U3.57 (I2C1_SMBA/I2S3_SD/SPI1_MOSI/SPI3_MOSI/TIM3_CH2/PB5)
- net KEY_A: now also U3.53 (PC12/I2S3_SD/SDIO_CK/SPI3_MOSI)
- net KEY_B: now also U3.2 (PC13/ANTI_TAMP/RTC_AF1)
- net KEY_C: now also U3.3 (PC14/RCC_OSC32_IN)
- net KEY_CW: now also U3.52 (PC11/ADC1_EXTI11/I2S3_ext_SD/SDIO_D3/SPI3_MISO)
- net KEY_D: now also U3.4 (PC15/ADC1_EXTI15/RCC_OSC32_OUT)
- net KEY_MENU: now also U3.40 (PC9/I2C3_SDA/I2S_CKIN/RCC_MCO_2/SDIO_D1/TIM3_CH4)
- net LCD_CE: now also U3.20 (ADC1_IN4/I2S3_WS/SPI1_NSS/SPI3_NSS/USART2_CK/PA4)
- net LCD_CLK: now also U3.21 (ADC1_IN5/SPI1_SCK/TIM2_CH1/TIM2_ETR/PA5)
- net LCD_DC: now also U3.22 (ADC1_IN6/SPI1_MISO/TIM1_BKIN/TIM3_CH1/PA6)
- net LCD_DIN: now also U3.23 (ADC1_IN7/SPI1_MOSI/TIM1_CH1N/TIM3_CH2/PA7)
- net LCD_LIGHT: now also U3.25 (PC5/ADC1_IN15)
- net LCD_RESET: now also U3.24 (PC4/ADC1_IN14)
- net LINE_OUT_LEFT_MCU: now also U3.16 (ADC1_IN2/TIM2_CH3/TIM5_CH3/TIM9_CH1/USART2_TX/PA2)
- net LINE_OUT_RIGHT_MCU: now also U3.17 (ADC1_IN3/TIM2_CH4/TIM5_CH4/TIM9_CH2/USART2_RX/PA3)
- net MCU_RESET: now also C29.1, U3.7 (NRST)
- net PTT_IN: now also U3.51 (PC10/I2S3_CK/SDIO_D2/SPI3_SCK)
- net Q_IN_M1: now also U3.58 (I2C1_SCL/TIM4_CH1/USART1_TX/PB6)
- net Q_IN_M2: now also U3.59 (I2C1_SDA/TIM4_CH2/USART1_RX/PB7)
- net S-metr: now also U3.8 (PC0/ADC1_IN10)
- net SWCLK: now also U3.49 (SYS_JTCK-SWCLK/PA14)
- net SWDIO: now also U3.46 (SYS_JTMS-SWDIO/PA13)
- net SWO: now also U3.55 (I2C2_SDA/I2S3_CK/SPI1_SCK/SPI3_SCK/SYS_JTDO-SWO/TIM2_CH2/PB3)
- net TX1: now also U3.41 (I2C3_SCL/RCC_MCO_1/TIM1_CH1/USART1_CK/USB_OTG_FS_SOF/PA8)
- net TX2: now also U3.50 (ADC1_EXTI15/I2S3_WS/SPI1_NSS/SPI3_NSS/SYS_JTDI/TIM2_CH1/TIM2_ETR/PA15)
- net UART_RX: now also U3.42 (I2C3_SMBA/TIM1_CH2/USART1_TX/USB_OTG_FS_VBUS/PA9)
- net UART_TX: now also U3.43 (TIM1_CH3/USART1_RX/USB_OTG_FS_ID/PA10)
- net USB_DM: now also U3.44 (ADC1_EXTI11/TIM1_CH4/USART1_CTS/USART6_TX/USB_OTG_FS_DM/PA11)
- net USB_DP: now also U3.45 (TIM1_ETR/USART1_RTS/USART6_RX/USB_OTG_FS_DP/PA12)
- net at Y1.1: now also C28.1, U3.5 (PH0/RCC_OSC_IN)
- net at Y1.2: now also C30.1, U3.6 (PH1/RCC_OSC_OUT)
- new net: C32.1, U3.30 (VCAP1)
- new net: R7.2, U3.31 (VSS)
- new net: R8.1, U3.47 (VSS)
Changed lines of the file:
@@
 LIBS:4ms-ic
 LIBS:Display
-LIBS:TRXklopik
-LIBS:stm32
-LIBS:switches
-LIBS:cmos4000
-LIBS:conn
+LIBS:Connector
+LIBS:Relay
 LIBS:LCSDR-cache
 EELAYER 25 0
@@
 Wire Wire Line
 	8600 4650 8250 4650
-Wire Wire Line
-	8900 5000 10000 4900
 Text GLabel 10000 3000 2    60   BiDi ~ 0
 SWDIO
@@
 Text GLabel 10000 4050 2    60   BiDi ~ 0
 SWO
-$Comp
-L STM32F401RCTx U19
-U 1 1 5DD6394C
-P 5950 3450
-F 0 "U19" H 3750 5375 50  0000 L BNN
-F 1 "STM32F401RCTx" H 8150 5375 50  0000 R BNN
-F 2 "LQFP64" H 8150 5325 50  0001 R TNN
-F 3 "" H 5950 3450 50  0001 C CNN
-	1    5950 3450
-	1    0    0    -1
-$EndComp
-$Comp
-L C_Small C120
-U 1 1 5DD63F21
-P 3250 2600
-F 0 "C120" H 3350 2650 50  0000 L CNN
-F 1 "100nF" H 3350 2550 50  0000 L CNN
-F 2 "" H 3250 2600 50  0001 C CNN
-F 3 "" H 3250 2600 50  0001 C CNN
-	1    3250 2600
-	1    0    0    -1
-$EndComp
 Wire Wire Line
 	3650 2450 3250 2450
 Wire Wire Line
 	3250 2450 3250 2500
-$Comp
-L R_Small R85
-U 1 1 5DD64E95
-P 5950 5700
-F 0 "R85" H 6000 5750 50  0000 L CNN
-F 1 "0*" H 6000 5650 50  0000 L CNN
-F 2 "" H 5950 5700 50  0001 C CNN
-F 3 "" H 5950 5700 50  0001 C CNN
-	1    5950 5700
-	1    0    0    -1
-$EndComp
-$Comp
-L R_Small R84
-U 1 1 5DD64F1C
-P 5850 5700
-F 0 "R84" H 5900 5650 50  0000 L CNN
-F 1 "0*" H 5900 5750 50  0000 L CNN
-F 2 "" H 5850 5700 50  0001 C CNN
-F 3 "" H 5850 5700 50  0001 C CNN
-	1    5850 5700
-	-1   0    0    1
-$EndComp
 $Comp
 L GND #PWR039
@@
 F 0 "Y1" H 2800 2800 50  0000 C CNN
 F 1 "20Mhz" H 2800 2500 50  0000 C CNN
-F 2 "" H 2800 2650 50  0001 C CNN
+F 2 "Crystals:Crystal_HC49-U_Vertical" H 2800 2650 50  0001 C CNN
 F 3 "" H 2800 2650 50  0001 C CNN
 	1    2800 2650
@@
 Wire Wire Line
 	2550 2950 3650 2950
-$Comp
-L C_Small C117
-U 1 1 5DD65463
-P 2550 3200
-F 0 "C117" H 2560 3270 50  0000 L CNN
-F 1 "C_Small" H 2560 3120 50  0000 L CNN
-F 2 "" H 2550 3200 50  0001 C CNN
-F 3 "" H 2550 3200 50  0001 C CNN
-	1    2550 3200
-	1    0    0    -1
-$EndComp
-$Comp
-L C_Small C119
-U 1 1 5DD65550
-P 3050 3200
-F 0 "C119" H 3060 3270 50  0000 L CNN
-F 1 "C_Small" H 3060 3120 50  0000 L CNN
-F 2 "" H 3050 3200 50  0001 C CNN
-F 3 "" H 3050 3200 50  0001 C CNN
-	1    3050 3200
-	1    0    0    -1
-$EndComp
 $Comp
 L GND #PWR042
@@
 	1    0    0    -1
 $EndComp
-$Comp
-L C_Small C118
-U 1 1 5DD65821
-P 2750 2000
-F 0 "C118" H 2850 2050 50  0000 L CNN
-F 1 "100nF" H 2850 1950 50  0000 L CNN
-F 2 "" H 2750 2000 50  0001 C CNN
-F 3 "" H 2750 2000 50  0001 C CNN
-	1    2750 2000
-	1    0    0    -1
-$EndComp
 Wire Wire Line
 	2550 1850 3650 1850
@@
 $EndComp
 $Comp
-L 24LC16 U17
-U 1 1 5DD65E9D
-P 1450 1400
-F 0 "U17" H 1200 1650 50  0000 C CNN
-F 1 "FM24CL16B" H 1500 1650 50  0000 L CNN
-F 2 "Housings_SOIC:SOIC-8_3.9x4.9mm_Pitch1.27mm" H 1500 1150 50  0001 L CNN
-F 3 "" H 1450 1300 50  0001 C CNN
-	1    1450 1400
-	1    0    0    -1
-$EndComp
-$Comp
 L GND #PWR045
 U 1 1 5DD66640
@@
 	1    0    0    -1
 $EndComp
-$Comp
-L C_Small C129
-U 1 1 5DD9FD31
-P 1200 950
-F 0 "C129" V 950 850 50  0000 L CNN
-F 1 "100nF" V 1050 850 50  0000 L CNN
-F 2 "" H 1200 950 50  0001 C CNN
-F 3 "" H 1200 950 50  0001 C CNN
-	1    1200 950
-	0    1    1    0
-$EndComp
-Wire Wire Line
-	1300 950  1450 950
+Wire Wire Line
+	1100 950  1450 950
 Wire Wire Line
 	1450 900  1450 1100
@@
 L GND #PWR048
 U 1 1 5DDA00B4
-P 1100 950
-F 0 "#PWR048" H 1100 700 50  0001 C CNN
-F 1 "GND" H 1100 800 50  0001 C CNN
-F 2 "" H 1100 950 50  0001 C CNN
-F 3 "" H 1100 950 50  0001 C CNN
-	1    1100 950
+P 900 950
+F 0 "#PWR048" H 900 700 50  0001 C CNN
+F 1 "GND" H 900 800 50  0001 C CNN
+F 2 "" H 900 950 50  0001 C CNN
+F 3 "" H 900 950 50  0001 C CNN
+	1    900  950
 	0    1    1    0
 $EndComp
@@
 	5750 1450 5750 1300
 Connection ~ 5750 1300
-$Comp
-L C_Small C130
-U 1 1 5DDA07EC
-P 6800 800
-F 0 "C130" H 6500 750 50  0000 L CNN
-F 1 "100nF" H 6450 850 50  0000 L CNN
-F 2 "" H 6800 800 50  0001 C CNN
-F 3 "" H 6800 800 50  0001 C CNN
-	1    6800 800
-	-1   0    0    1
-$EndComp
-$Comp
-L C_Small C131
-U 1 1 5DDA0BB8
-P 7300 800
-F 0 "C131" H 7000 750 50  0000 L CNN
-F 1 "100nF" H 6950 850 50  0000 L CNN
-F 2 "" H 7300 800 50  0001 C CNN
-F 3 "" H 7300 800 50  0001 C CNN
-	1    7300 800
-	-1   0    0    1
-$EndComp
-$Comp
-L C_Small C132
-U 1 1 5DDA0C05
-P 7800 800
-F 0 "C132" H 7500 750 50  0000 L CNN
-F 1 "100nF" H 7450 850 50  0000 L CNN
-F 2 "" H 7800 800 50  0001 C CNN
-F 3 "" H 7800 800 50  0001 C CNN
-	1    7800 800
-	-1   0    0    1
-$EndComp
 $Comp
 L +3V3 #PWR050
@@
 	8250 4450 8800 4450
 Wire Wire Line
-	8800 4450 8800 5150
-Wire Wire Line
-	8800 5150 10000 5050
-Wire Wire Line
-	8900 5000 8900 4350
-Wire Wire Line
 	8900 4350 8250 4350
 Text GLabel 10000 4700 2    60   Output ~ 0
@@
 	8250 4250 9000 4250
 Wire Wire Line
-	9000 4250 9000 4850
-Wire Wire Line
-	10000 4550 9100 4700
-Wire Wire Line
-	9100 4700 9100 4150
-Wire Wire Line
 	9100 4150 8250 4150
 Wire Wire Line
 	8250 4050 9200 4050
 Wire Wire Line
-	9200 4050 9200 4550
-Wire Wire Line
-	9200 4550 10000 4400
-Wire Wire Line
-	9000 4850 10000 4700
-Wire Wire Line
 	8250 3950 9300 3950
-Wire Wire Line
-	9300 3950 9300 4400
-Wire Wire Line
-	9300 4400 10000 4250
 Wire Wire Line
 	9400 3850 8250 3850
@@
 	9500 3750 8250 3750
 Wire Wire Line
-	10000 5250 8700 5300
-Wire Wire Line
-	8700 5300 8700 4550
-Wire Wire Line
 	8700 4550 8250 4550
 Text GLabel 10000 1950 2    60   Output ~ 0
@@
 Wire Wire Line
 	9400 4050 10000 4050
+$Comp
+L C_Small C28
+U 1 1 5DDF67B4
+P 2550 3200
+F 0 "C28" H 2650 3250 50  0000 L CNN
+F 1 "22" H 2650 3150 50  0000 L CNN
+F 2 "UI:C_1206_0603" H 2550 3200 50  0001 C CNN
+F 3 "" H 2550 3200 50  0001 C CNN
+	1    2550 3200
+	1    0    0    -1
+$EndComp
+$Comp
+L C_Small C30
+U 1 1 5DDF6854
+P 3050 3200
+F 0 "C30" H 3150 3250 50  0000 L CNN
+F 1 "22" H 3150 3150 50  0000 L CNN
+F 2 "UI:C_1206_0603" H 3050 3200 50  0001 C CNN
+F 3 "" H 3050 3200 50  0001 C CNN
+	1    3050 3200
+	1    0    0    -1
+$EndComp
+$Comp
+L C_Small C32
+U 1 1 5DDF6B89
+P 3250 2600
+F 0 "C32" H 3350 2650 50  0000 L CNN
+F 1 "100nF" H 3350 2550 50  0000 L CNN
+F 2 "UI:C_1206_0603" H 3250 2600 50  0001 C CNN
+F 3 "" H 3250 2600 50  0001 C CNN
+	1    3250 2600
+	1    0    0    -1
+$EndComp
+$Comp
+L C_Small C29
+U 1 1 5DDF6C62
+P 2750 2000
+F 0 "C29" H 2850 2050 50  0000 L CNN
+F 1 "100nF" H 2850 1950 50  0000 L CNN
+F 2 "UI:C_1206_0603" H 2750 2000 50  0001 C CNN
+F 3 "" H 2750 2000 50  0001 C CNN
+	1    2750 2000
+	1    0    0    -1
+$EndComp
+$Comp
+L C_Small C33
+U 1 1 5DDF6E50
+P 6800 800
+F 0 "C33" H 6500 750 50  0000 L CNN
+F 1 "100nF" H 6450 850 50  0000 L CNN
+F 2 "UI:C_1206_0603" H 6800 800 50  0001 C CNN
+F 3 "" H 6800 800 50  0001 C CNN
+	1    6800 800
+	-1   0    0    1
+$EndComp
+$Comp
+L C_Small C34
+U 1 1 5DDF6F13
+P 7300 800
+F 0 "C34" H 7000 750 50  0000 L CNN
+F 1 "100nF" H 6950 850 50  0000 L CNN
+F 2 "UI:C_1206_0603" H 7300 800 50  0001 C CNN
+F 3 "" H 7300 800 50  0001 C CNN
+	1    7300 800
+	-1   0    0    1
+$EndComp
+$Comp
+L C_Small C35
+U 1 1 5DDF6F66
+P 7800 800
+F 0 "C35" H 7500 750 50  0000 L CNN
+F 1 "100nF" H 7450 850 50  0000 L CNN
+F 2 "UI:C_1206_0603" H 7800 800 50  0001 C CNN
+F 3 "" H 7800 800 50  0001 C CNN
+	1    7800 800
+	-1   0    0    1
+$EndComp
+$Comp
+L C_Small C27
+U 1 1 5DDF7102
+P 1000 950
+F 0 "C27" V 750 850 50  0000 L CNN
+F 1 "100nF" V 850 850 50  0000 L CNN
+F 2 "UI:C_1206_0603" H 1000 950 50  0001 C CNN
+F 3 "" H 1000 950 50  0001 C CNN
+	1    1000 950
+	0    1    1    0
+$EndComp
+$Comp
+L R_Small R7
+U 1 1 5DDF73A0
+P 5850 5700
+F 0 "R7" H 5900 5650 50  0000 L CNN
+F 1 "0*" H 5900 5750 50  0000 L CNN
+F 2 "UI:R_1206_0603" H 5850 5700 50  0001 C CNN
+F 3 "" H 5850 5700 50  0001 C CNN
+	1    5850 5700
+	-1   0    0    1
+$EndComp
+$Comp
+L R_Small R8
+U 1 1 5DDF7436
+P 5950 5700
+F 0 "R8" H 6000 5750 50  0000 L CNN
+F 1 "0*" H 6000 5650 50  0000 L CNN
+F 2 "UI:R_1206_0603" H 5950 5700 50  0001 C CNN
+F 3 "" H 5950 5700 50  0001 C CNN
+	1    5950 5700
+	1    0    0    -1
+$EndComp
+$Comp
+L STM32F401RCTx U3
+U 1 1 5DDFBAAA
+P 5950 3450
+F 0 "U3" H 3750 5375 50  0000 L BNN
+F 1 "STM32F401RCTx" H 8150 5375 50  0000 R BNN
+F 2 "Housings_QFP:LQFP-64_10x10mm_Pitch0.5mm" H 8150 5325 50  0001 R TNN
+F 3 "" H 5950 3450 50  0001 C CNN
+	1    5950 3450
+	1    0    0    -1
+$EndComp
+$Comp
+L 24LC16 U2
+U 1 1 5DDFBE63
+P 1450 1400
+F 0 "U2" H 1200 1650 50  0000 C CNN
+F 1 "FM24CL16B" H 1500 1650 50  0000 L CNN
+F 2 "Housings_SOIC:SOIC-8_3.9x4.9mm_Pitch1.27mm" H 1500 1150 50  0001 L CNN
+F 3 "" H 1450 1300 50  0001 C CNN
+	1    1450 1400
+	1    0    0    -1
+$EndComp
+Wire Wire Line
+	9300 3950 9300 4250
+Wire Wire Line
+	9300 4250 10000 4250
+Wire Wire Line
+	9200 4050 9200 4400
+Wire Wire Line
+	9200 4400 10000 4400
+Wire Wire Line
+	9100 4150 9100 4550
+Wire Wire Line
+	9100 4550 10000 4550
+Wire Wire Line
+	9000 4250 9000 4700
+Wire Wire Line
+	9000 4700 10000 4700
+Wire Wire Line
+	8900 4350 8900 4900
+Wire Wire Line
+	8900 4900 10000 4900
+Wire Wire Line
+	8800 4450 8800 5050
+Wire Wire Line
+	8800 5050 10000 5050
+Wire Wire Line
+	10000 5250 8700 5250
+Wire Wire Line
+	8700 5250 8700 4550
 $EndSCHEMATC

Commit message: PCB update
Connections:
- net I2C_SCL: no longer U3.61 (I2C1_SCL/SDIO_D4/TIM10_CH1/TIM4_CH3/PB8)
- net I2C_SDA: no longer U3.62 (I2C1_SDA/I2S2_WS/SDIO_D5/SPI2_NSS/TIM11_CH1/TIM4_CH4/PB9)
- net LINE_OUT_LEFT_MCU: no longer U3.16 (ADC1_IN2/TIM2_CH3/TIM5_CH3/TIM9_CH1/USART2_TX/PA2)
- net LINE_OUT_RIGHT_MCU: no longer U3.17 (ADC1_IN3/TIM2_CH4/TIM5_CH4/TIM9_CH2/USART2_RX/PA3)
- new net I2C_SCL_MCU: U3.61 (I2C1_SCL/SDIO_D4/TIM10_CH1/TIM4_CH3/PB8)
- new net I2C_SDA_MCU: U3.62 (I2C1_SDA/I2S2_WS/SDIO_D5/SPI2_NSS/TIM11_CH1/TIM4_CH4/PB9)
Changed lines of the file:
@@
 I2S_LRCK
 Text GLabel 10000 4900 2    60   Output ~ 0
-I2C_SCL
+I2C_SCL_MCU
 Text GLabel 10000 5050 2    60   BiDi ~ 0
-I2C_SDA
+I2C_SDA_MCU
 Wire Wire Line
 	8250 4950 8300 4950
@@
 	3250 2450 3250 2500
 $Comp
-L GND #PWR039
+L GND #PWR035
 U 1 1 5DD64FC0
 P 5900 5900
-F 0 "#PWR039" H 5900 5650 50  0001 C CNN
+F 0 "#PWR035" H 5900 5650 50  0001 C CNN
 F 1 "GND" H 5900 5750 50  0001 C CNN
 F 2 "" H 5900 5900 50  0001 C CNN
@@
 	5950 5350 5950 5600
 $Comp
-L GND #PWR040
+L GND #PWR036
 U 1 1 5DD650F1
 P 6150 5450
-F 0 "#PWR040" H 6150 5200 50  0001 C CNN
+F 0 "#PWR036" H 6150 5200 50  0001 C CNN
 F 1 "GND" H 6150 5300 50  0001 C CNN
 F 2 "" H 6150 5450 50  0001 C CNN
@@
 Connection ~ 6150 5400
 $Comp
-L GND #PWR041
+L GND #PWR037
 U 1 1 5DD65332
 P 3250 2700
-F 0 "#PWR041" H 3250 2450 50  0001 C CNN
+F 0 "#PWR037" H 3250 2450 50  0001 C CNN
 F 1 "GND" H 3250 2550 50  0001 C CNN
 F 2 "" H 3250 2700 50  0001 C CNN
@@
 	2550 2950 3650 2950
 $Comp
-L GND #PWR042
+L GND #PWR038
 U 1 1 5DD65598
 P 3050 3300
-F 0 "#PWR042" H 3050 3050 50  0001 C CNN
+F 0 "#PWR038" H 3050 3050 50  0001 C CNN
 F 1 "GND" H 3050 3150 50  0001 C CNN
 F 2 "" H 3050 3300 50  0001 C CNN
@@
 $EndComp
 $Comp
-L GND #PWR043
+L GND #PWR039
 U 1 1 5DD655DB
 P 2550 3300
-F 0 "#PWR043" H 2550 3050 50  0001 C CNN
+F 0 "#PWR039" H 2550 3050 50  0001 C CNN
 F 1 "GND" H 2550 3150 50  0001 C CNN
 F 2 "" H 2550 3300 50  0001 C CNN
@@
 	2750 1850 2750 1900
 $Comp
-L GND #PWR044
+L GND #PWR040
 U 1 1 5DD65924
 P 2750 2100
-F 0 "#PWR044" H 2750 1850 50  0001 C CNN
+F 0 "#PWR040" H 2750 1850 50  0001 C CNN
 F 1 "GND" H 2750 1950 50  0001 C CNN
 F 2 "" H 2750 2100 50  0001 C CNN
@@
 $EndComp
 $Comp
-L GND #PWR045
+L GND #PWR041
 U 1 1 5DD66640
 P 1450 1700
-F 0 "#PWR045" H 1450 1450 50  0001 C CNN
+F 0 "#PWR041" H 1450 1450 50  0001 C CNN
 F 1 "GND" H 1450 1550 50  0001 C CNN
 F 2 "" H 1450 1700 50  0001 C CNN
@@
 $EndComp
 $Comp
-L GND #PWR046
+L GND #PWR042
 U 1 1 5DD667F8
 P 1900 1550
-F 0 "#PWR046" H 1900 1300 50  0001 C CNN
+F 0 "#PWR042" H 1900 1300 50  0001 C CNN
 F 1 "GND" H 1900 1400 50  0001 C CNN
 F 2 "" H 1900 1550 50  0001 C CNN
@@
 	2100 1450 2300 1450
 $Comp
-L +3V3 #PWR047
+L +3V3 #PWR043
 U 1 1 5DD9FC90
 P 1450 900
-F 0 "#PWR047" H 1450 750 50  0001 C CNN
+F 0 "#PWR043" H 1450 750 50  0001 C CNN
 F 1 "+3V3" H 1450 1050 50  0000 C CNN
 F 2 "" H 1450 900 50  0001 C CNN
@@
 Connection ~ 1450 950
 $Comp
-L GND #PWR048
+L GND #PWR044
 U 1 1 5DDA00B4
 P 900 950
-F 0 "#PWR048" H 900 700 50  0001 C CNN
+F 0 "#PWR044" H 900 700 50  0001 C CNN
 F 1 "GND" H 900 800 50  0001 C CNN
 F 2 "" H 900 950 50  0001 C CNN
@@
 $EndComp
 $Comp
-L +3V3 #PWR049
+L +3V3 #PWR045
 U 1 1 5DDA012B
 P 5550 1300
-F 0 "#PWR049" H 5550 1150 50  0001 C CNN
+F 0 "#PWR045" H 5550 1150 50  0001 C CNN
 F 1 "+3V3" V 5550 1550 50  0000 C CNN
 F 2 "" H 5550 1300 50  0001 C CNN
@@
 Connection ~ 5750 1300
 $Comp
-L +3V3 #PWR050
+L +3V3 #PWR046
 U 1 1 5DDA0C93
 P 6600 650
-F 0 "#PWR050" H 6600 500 50  0001 C CNN
+F 0 "#PWR046" H 6600 500 50  0001 C CNN
 F 1 "+3V3" V 6600 900 50  0000 C CNN
 F 2 "" H 6600 650 50  0001 C CNN
@@
 Connection ~ 6800 650
 $Comp
-L GND #PWR051
+L GND #PWR047
 U 1 1 5DDA0E68
 P 6800 900
-F 0 "#PWR051" H 6800 650 50  0001 C CNN
+F 0 "#PWR047" H 6800 650 50  0001 C CNN
 F 1 "GND" H 6800 750 50  0001 C CNN
 F 2 "" H 6800 900 50  0001 C CNN
@@
 $EndComp
 $Comp
-L GND #PWR052
+L GND #PWR048
 U 1 1 5DDA0EDC
 P 7300 900
-F 0 "#PWR052" H 7300 650 50  0001 C CNN
+F 0 "#PWR048" H 7300 650 50  0001 C CNN
 F 1 "GND" H 7300 750 50  0001 C CNN
 F 2 "" H 7300 900 50  0001 C CNN
@@
 $EndComp
 $Comp
-L GND #PWR053
+L GND #PWR049
 U 1 1 5DDA0F4B
 P 7800 900
-F 0 "#PWR053" H 7800 650 50  0001 C CNN
+F 0 "#PWR049" H 7800 650 50  0001 C CNN
 F 1 "GND" H 7800 750 50  0001 C CNN
 F 2 "" H 7800 900 50  0001 C CNN
@@
 MCU_RESET
 Connection ~ 2750 1850
-Text GLabel 10000 950  2    60   Output ~ 0
-LINE_OUT_LEFT_MCU
 Wire Wire Line
 	8250 4450 8800 4450
@@
 Wire Wire Line
 	2250 5800 2050 5800
-Text GLabel 10000 1100 2    60   Output ~ 0
-LINE_OUT_RIGHT_MCU
 Wire Wire Line
 	8250 3650 9600 3650
@@
 	8250 3350 10000 3350
 Wire Wire Line
-	8250 2050 8550 2050
-Wire Wire Line
-	8650 2150 8250 2150
-Wire Wire Line
 	8250 2250 8750 2250
 Wire Wire Line
@@
 	8750 1300 10000 1300
 Wire Wire Line
-	10000 1100 8650 1100
-Wire Wire Line
-	8650 1100 8650 2150
-Wire Wire Line
-	10000 950  8550 950
-Wire Wire Line
-	8550 950  8550 2050
-Wire Wire Line
 	8450 1950 8450 750
 Wire Wire Line
@@
 	9650 3000 10000 3000
 $Comp
-L GND #PWR054
+L GND #PWR050
 U 1 1 5DDFAF2B
 P 3650 2050
-F 0 "#PWR054" H 3650 1800 50  0001 C CNN
+F 0 "#PWR050" H 3650 1800 50  0001 C CNN
 F 1 "GND" H 3650 1900 50  0001 C CNN
 F 2 "" H 3650 2050 50  0001 C CNN
@@
 Wire Wire Line
 	8700 5250 8700 4550
+Text GLabel 10000 950  2    60   Output ~ 0
+LINE_OUT_LEFT_MCU
+Text GLabel 10000 1100 2    60   Output ~ 0
+LINE_OUT_RIGHT_MCU
 $EndSCHEMATC
