File: PCB/ST32_SDR/_saved_syntez.sch (KiCad schematic (older format))
At the start: 12 parts, among them U1 SI5351A, Y2 Crystal

Commit message: PCB update
Parts:
- gave numbers to parts that had none: 2
Connections:
- net BAND0: now also RN3.4 (R4.1); no longer RN3.1 (R1.1)
- net BAND1: now also RN3.3 (R3.1); no longer RN3.2 (R2.1)
- net BAND2: now also RN3.2 (R2.1); no longer RN3.3 (R3.1)
- net BAND3: now also RN3.1 (R1.1); no longer RN3.4 (R4.1)
Changed lines of the file:
@@
 	3550 1500 3550 2250
 $Comp
-L +3V3 #PWR01
+L +3V3 #PWR2
 U 1 1 5DDEDF62
 P 3550 1500
-F 0 "#PWR01" H 3550 1350 50  0001 C CNN
+F 0 "#PWR2" H 3550 1350 50  0001 C CNN
 F 1 "+3V3" H 3550 1640 50  0000 C CNN
 F 2 "" H 3550 1500 50  0001 C CNN
@@
 	3000 2900 2550 2900
 $Comp
-L GND #PWR02
+L GND #PWR1
 U 1 1 5DDEE4A0
 P 3150 1800
-F 0 "#PWR02" H 3150 1550 50  0001 C CNN
+F 0 "#PWR1" H 3150 1550 50  0001 C CNN
 F 1 "GND" H 3150 1650 50  0001 C CNN
 F 2 "" H 3150 1800 50  0001 C CNN
@@
 $EndComp
 $Comp
-L GND #PWR03
+L GND #PWR3
 U 1 1 5DDEE4E1
 P 5000 2450
-F 0 "#PWR03" H 5000 2200 50  0001 C CNN
+F 0 "#PWR3" H 5000 2200 50  0001 C CNN
 F 1 "GND" H 5000 2300 50  0001 C CNN
 F 2 "" H 5000 2450 50  0001 C CNN
@@
 $EndComp
 $Comp
-L +3V3 #PWR04
+L +3V3 #PWR4
 U 1 1 5DDEE519
 P 5000 2550
-F 0 "#PWR04" H 5000 2400 50  0001 C CNN
+F 0 "#PWR4" H 5000 2400 50  0001 C CNN
 F 1 "+3V3" V 5000 2800 50  0000 C CNN
 F 2 "" H 5000 2550 50  0001 C CNN
@@
 Connection ~ 6100 1100
 $Comp
-L GND #PWR05
+L GND #PWR5
 U 1 1 5DDEEBF2
 P 6100 1400
-F 0 "#PWR05" H 6100 1150 50  0001 C CNN
+F 0 "#PWR5" H 6100 1150 50  0001 C CNN
 F 1 "GND" H 6100 1250 50  0001 C CNN
 F 2 "" H 6100 1400 50  0001 C CNN
@@
 $EndComp
 $Comp
-L GND #PWR06
+L GND #PWR6
 U 1 1 5DDEEC35
 P 6100 2150
-F 0 "#PWR06" H 6100 1900 50  0001 C CNN
+F 0 "#PWR6" H 6100 1900 50  0001 C CNN
 F 1 "GND" H 6100 2000 50  0001 C CNN
 F 2 "" H 6100 2150 50  0001 C CNN
@@
 	6100 2650 6100 2750
 $Comp
-L GND #PWR07
+L GND #PWR7
 U 1 1 5DDEECF7
 P 6100 2950
-F 0 "#PWR07" H 6100 2700 50  0001 C CNN
+F 0 "#PWR7" H 6100 2700 50  0001 C CNN
 F 1 "GND" H 6100 2800 50  0001 C CNN
 F 2 "" H 6100 2950 50  0001 C CNN
@@
 	0    1    1    0
 $EndComp
-Text GLabel 2850 4250 0    60   Input ~ 0
+Text GLabel 2750 4850 0    60   Input ~ 0
 BAND0
 Wire Wire Line
 	3000 4400 3200 4400
-Text GLabel 2850 4450 0    60   Input ~ 0
+Text GLabel 2750 4650 0    60   Input ~ 0
 BAND1
 Wire Wire Line
 	2900 4500 3200 4500
-Text GLabel 2850 4650 0    60   Input ~ 0
+Text GLabel 2750 4450 0    60   Input ~ 0
 BAND2
 Wire Wire Line
-	2850 4450 2900 4450
+	2750 4450 2900 4450
 Wire Wire Line
 	2900 4450 2900 4500
 Wire Wire Line
-	2850 4650 2900 4650
+	2750 4650 2900 4650
 Wire Wire Line
 	2900 4650 2900 4600
 Wire Wire Line
 	2900 4600 3200 4600
-Text GLabel 2850 4850 0    60   Input ~ 0
+Text GLabel 2750 4250 0    60   Input ~ 0
 BAND3
 Wire Wire Line
-	2850 4250 3000 4250
+	2750 4250 3000 4250
 Wire Wire Line
 	3000 4250 3000 4400
 Wire Wire Line
-	2850 4850 3000 4850
+	2750 4850 3000 4850
 Wire Wire Line
 	3000 4850 3000 4700
@@
 I2C_SDA_MCU
 $Comp
-L R_Small R?
+L R_Small R22
 U 1 1 5DE23CAB
 P 1550 1050
-F 0 "R?" V 1750 1050 50  0000 L CNN
+F 0 "R22" V 1750 1050 50  0000 L CNN
 F 1 "56" V 1650 1050 50  0000 L CNN
 F 2 "" H 1550 1050 50  0001 C CNN
@@
 $EndComp
 $Comp
-L R_Small R?
+L R_Small R23
 U 1 1 5DE23D38
 P 1550 1300
-F 0 "R?" V 1450 1300 50  0000 L CNN
+F 0 "R23" V 1450 1300 50  0000 L CNN
 F 1 "56" V 1350 1300 50  0000 L CNN
 F 2 "" H 1550 1300 50  0001 C CNN
