File: PCB/ST32_SDR/AUDIO_OUT.sch (KiCad schematic (older format))
At the start: 23 parts, among them J1 Audio-Jack-3_2Switches, J3 Audio-Jack-3_2Switches, U13 4053, U16 WM8731_alt

Commit message: Schematics update
Parts:
- J1: value Audio-Jack-3_2Switches -> MIC
Connections:
- net I2C2_SCL: no longer R77.2
- net I2S_SCLK: now reaches R80.2
- net I2S_SDO: now reaches R81.2
- net I2S_LRCK: now reaches R82.2
- net I2S_SDI: now reaches R83.2
- new net I2S_MCLK: R77.2
Changed lines of the file:
@@
 LIBS:contrib
 LIBS:LCSDR
+LIBS:Logic_74xx
+LIBS:Logic_CMOS_4000
 LIBS:4ms-ic
-LIBS:stm32
+LIBS:Connector
+LIBS:Display
+LIBS:TRXklopik
 LIBS:LCSDR-cache
 EELAYER 25 0
@@
 $Descr A4 11693 8268
 encoding utf-8
-Sheet 3 5
+Sheet 3 6
 Title ""
 Date ""
@@
 	4200 2350 4550 2350
 $Comp
-L GND #PWR157
+L GND #PWR0157
 U 1 1 5DD23C63
 P 4150 2750
-F 0 "#PWR157" H 4150 2500 50  0001 C CNN
+F 0 "#PWR0157" H 4150 2500 50  0001 C CNN
 F 1 "GND" H 4150 2600 50  0001 C CNN
 F 2 "" H 4150 2750 50  0001 C CNN
@@
 $EndComp
 $Comp
-L GND #PWR166
+L GND #PWR0158
 U 1 1 5DD2681A
 P 8650 2950
-F 0 "#PWR166" H 8650 2700 50  0001 C CNN
+F 0 "#PWR0158" H 8650 2700 50  0001 C CNN
 F 1 "GND" H 8650 2800 50  0001 C CNN
 F 2 "" H 8650 2950 50  0001 C CNN
@@
 P 6400 3850
 F 0 "J3" H 6400 4140 50  0000 C CNN
-F 1 "Audio-Jack-3_2Switches" H 6250 3650 50  0000 L CNN
+F 1 "Audio-Jack-3_2Switches" H 6250 3650 50  0001 L CNN
 F 2 "LCSDR:audio_jack_3_5mm_PJ307" H 6650 3950 50  0001 C CNN
 F 3 "" H 6650 3950 50  0001 C CNN
@@
 	6850 3400 7150 3400
 $Comp
-L GND #PWR160
+L GND #PWR0159
 U 1 1 5DD26DA0
 P 6200 4050
-F 0 "#PWR160" H 6200 3800 50  0001 C CNN
+F 0 "#PWR0159" H 6200 3800 50  0001 C CNN
 F 1 "GND" H 6200 3900 50  0001 C CNN
 F 2 "" H 6200 4050 50  0001 C CNN
@@
 U 1 1 5DD26E6D
 P 5050 4700
-F 0 "J1" H 5050 4990 50  0000 C CNN
-F 1 "Audio-Jack-3_2Switches" H 4900 4500 50  0000 L CNN
+F 0 "J1" H 5000 5000 50  0000 C CNN
+F 1 "MIC" H 4950 4500 50  0000 L CNN
 F 2 "" H 5300 4800 50  0001 C CNN
 F 3 "" H 5300 4800 50  0001 C CNN
@@
 Connection ~ 8650 1800
 $Comp
-L GND #PWR164
+L GND #PWR0160
 U 1 1 5DD27D3B
 P 8550 2000
-F 0 "#PWR164" H 8550 1750 50  0001 C CNN
+F 0 "#PWR0160" H 8550 1750 50  0001 C CNN
 F 1 "GND" H 8550 1850 50  0001 C CNN
 F 2 "" H 8550 2000 50  0001 C CNN
@@
 	8850 3400 8550 3400
 Wire Wire Line
-	9700 3350 9900 3350
+	9700 3350 10100 3350
 $Comp
 L CP_Small C116
@@
 $EndComp
 $Comp
-L GND #PWR162
+L GND #PWR0161
 U 1 1 5DD2888E
 P 7150 1900
-F 0 "#PWR162" H 7150 1650 50  0001 C CNN
+F 0 "#PWR0161" H 7150 1650 50  0001 C CNN
 F 1 "GND" H 7150 1750 50  0001 C CNN
 F 2 "" H 7150 1900 50  0001 C CNN
@@
 $EndComp
 $Comp
-L GND #PWR163
+L GND #PWR0162
 U 1 1 5DD288DB
 P 7150 2200
-F 0 "#PWR163" H 7150 1950 50  0001 C CNN
+F 0 "#PWR0162" H 7150 1950 50  0001 C CNN
 F 1 "GND" H 7150 2050 50  0001 C CNN
 F 2 "" H 7150 2200 50  0001 C CNN
@@
 	6750 2150 5850 2150
 $Comp
-L GND #PWR161
+L GND #PWR0163
 U 1 1 5DD292E5
 P 6300 2400
-F 0 "#PWR161" H 6300 2150 50  0001 C CNN
+F 0 "#PWR0163" H 6300 2150 50  0001 C CNN
 F 1 "GND" H 6300 2250 50  0001 C CNN
 F 2 "" H 6300 2400 50  0001 C CNN
@@
 	5850 2150 5850 2200
 $Comp
-L GND #PWR159
+L GND #PWR0164
 U 1 1 5DD29619
 P 5850 2400
-F 0 "#PWR159" H 5850 2150 50  0001 C CNN
+F 0 "#PWR0164" H 5850 2150 50  0001 C CNN
 F 1 "GND" H 5850 2250 50  0001 C CNN
 F 2 "" H 5850 2400 50  0001 C CNN
@@
 Connection ~ 9100 2700
 $Comp
-L +3.3V #PWR167
+L +3.3V #PWR0165
 U 1 1 5DD2A31B
 P 8950 1950
-F 0 "#PWR167" H 8950 1800 50  0001 C CNN
+F 0 "#PWR0165" H 8950 1800 50  0001 C CNN
 F 1 "+3.3V" H 8950 2090 50  0000 C CNN
 F 2 "" H 8950 1950 50  0001 C CNN
@@
 Connection ~ 8950 2000
 $Comp
-L +3.3V #PWR165
+L +3.3V #PWR0166
 U 1 1 5DD2A6BD
 P 8650 1700
-F 0 "#PWR165" H 8650 1550 50  0001 C CNN
+F 0 "#PWR0166" H 8650 1550 50  0001 C CNN
 F 1 "+3.3V" H 8650 1840 50  0000 C CNN
 F 2 "" H 8650 1700 50  0001 C CNN
@@
 	8950 3950 9500 3950
 $Comp
-L GND #PWR158
+L GND #PWR0167
 U 1 1 5DD2B06D
 P 4850 4900
-F 0 "#PWR158" H 4850 4650 50  0001 C CNN
+F 0 "#PWR0167" H 4850 4650 50  0001 C CNN
 F 1 "GND" H 4850 4750 50  0001 C CNN
 F 2 "" H 4850 4900 50  0001 C CNN
@@
 	9900 2600 9700 2600
 Text GLabel 10050 2300 2    60   Input ~ 0
-I2C2_SCL
+I2S_MCLK
 Wire Wire Line
 	10050 2300 9700 2300
+Text GLabel 10100 3950 2    60   BiDi ~ 0
+I2S_LRCK
+Text GLabel 10100 3350 2    60   BiDi ~ 0
+I2S_SCLK
+Wire Wire Line
+	9700 3950 10100 3950
+Text GLabel 10100 3650 2    60   BiDi ~ 0
+I2S_SDO
+Wire Wire Line
+	10100 3650 9700 3650
+Text GLabel 10100 4250 2    60   BiDi ~ 0
+I2S_SDI
+Wire Wire Line
+	9700 4250 10100 4250
 $EndSCHEMATC

Commit message: update schematics
Parts:
- removed C112, C113: 2.2uF, symbol CP_Small
- removed C114: CP_Small, symbol CP_Small
- removed C99: 4.7uF, symbol CP_Small
- removed L27, L28: L_Small, symbol L_Small
- removed R51, R55: 10k, symbol R_Small
- removed R80, R81, R82, R83: 100, symbol R_Small
- removed U13: 4053, symbol 4053
- added C10, C11, C12, C13, C8, C9: 470nF, symbol C_Small
- added C14, C15, C17, C19, C95: 1uF, symbol CP_Small
- added C16, C21, C7: 100nF, symbol C_Small
- added C18, C20, C5, C6: 1nF, symbol C_Small
- added C75, C76: 2.2uF, symbol CP_Small
- added C94: 220, symbol C_Small
- added D1: LL4148, symbol D_Small
- added J4: LINEIN, symbol Audio-Jack-3_2Switches
- added R105: 680, symbol R_Small
- added R4: 4.7k, symbol R_Small
- added R5, R6: 0*, symbol R_Small
- added RN4, RN5, RN7: 47, symbol R_Pack04
- added RN6: 4.7k, symbol R_Pack04
- added U13, U20: 4066, symbol 4066
- J1: value MIC -> MIC_PTT
Connections:
- net +3V3: now also U16.14 (AVDD), U16.8 (HPVDD), R4.1, R6.1
- net GND: now also C16.2, C18.2, C20.2, C21.2, C5.2, C6.2, C7.2, C94.2, J4.3, RN6.2 (R2.1), RN6.4 (R4.1), U13.7 (V-), U13.7 (V-), U13.7 (V-), U13.7 (V-), U20.7 (V-), U20.7 (V-)
- net I2S_LRCK: now also RN7.6 (R3.2)
- net I2S_SCLK: now also RN7.8 (R1.2)
- net I2S_SDI: now also RN7.5 (R4.2)
- net I2S_SDO: now also RN7.7 (R2.2)
- net at U16.10 (RHPOUT): now also C19.1; no longer J3.4
- net LINE_OUT_LEFT: now reaches U16.12 (LOUT)
- net LINE_OUT_LEFT: now also C12.2
- net LINE_OUT_RIGHT: now reaches U16.13 (ROUT)
- net LINE_OUT_RIGHT: now also C13.2
- net MIC_BIAS: now reaches U16.17 (MICBIAS)
- net MIC_BIAS: now also R105.2
- net MIC_IN: now reaches U16.18 (MICIN)
- net MIC_IN: now also C95.1
- net LINE_IN_RIGHT: now reaches U16.19 (RLINEIN)
- net LINE_IN_RIGHT: now also C15.1
- net LINE_IN_LEFT: now reaches U16.20 (LLINEIN)
- net LINE_IN_LEFT: now also C14.1
- net at U16.3 (BCLK): now also RN7.1 (R1.1)
- net at U16.4 (DACDAT): now also RN7.2 (R2.1)
- net at U16.5 (DACLRC), U16.7 (ADCLRC): now also RN7.3 (R3.1)
- net at U16.6 (ADCDAT): now also RN7.4 (R4.1)
- net at U16.9 (LHPOUT): now also C17.1; no longer J3.5
- net at J3.1: now also J3.4, C19.2, C20.1
- net at J3.2: now also J3.5, C17.2, C18.1
- net at J1.1, J1.4: now also C94.1, C95.2, R105.1; no longer J1.2, J1.5
- new net: D1.1 (K), J1.2, J1.5
- new net: C10.2, U13.1 (I/O)
- new net: RN5.8 (R1.2), U13.13 (ON)
- new net: C14.2, U13.2 (O/I), U13.3 (O/I)
- new net: C5.1, J4.1, J4.4, RN6.3 (R3.1)
- new net: C6.1, J4.2, J4.5, RN6.1 (R1.1)
- new net: C75.1, U13.4 (I/O)
- new net: RN5.7 (R2.2), U13.5 (ON)
- new net: C76.1, U13.11 (I/O)
- new net: C76.2, RN6.5 (R4.2), RN6.6 (R3.2)
- new net: RN5.6 (R3.2), U13.6 (ON)
- new net: C11.2, U13.8 (I/O)
- new net: C15.2, U13.10 (O/I), U13.9 (O/I)
- new net: C75.2, RN6.7 (R2.2), RN6.8 (R1.2)
- new net: C13.1, U20.3 (O/I)
- new net: C9.2, U20.4 (I/O)
- new net: RN4.7 (R2.2), U20.5 (ON)
- new net: RN5.5 (R4.2), U13.12 (ON)
- new net: C8.2, U20.1 (I/O)
- new net: RN4.8 (R1.2), U20.13 (ON)
- new net: C12.1, U20.2 (O/I)
- new net +9VA: R5.1
- new net I_IN: C10.1
- new net I_IN_M1: RN5.1 (R1.1)
- new net I_IN_M2: RN5.2 (R2.1)
- new net I_OUT: C8.1
- new net LINE_OUT_LEFT_MCU: RN4.1 (R1.1)
- new net LINE_OUT_RIGHT_MCU: RN4.2 (R2.1)
- new net PTTIN: C7.1, D1.2 (A), R4.2
- new net Q_IN: C11.1
- new net Q_IN_M1: RN5.3 (R3.1)
- new net Q_IN_M2: RN5.4 (R4.1)
- new net Q_OUT: C9.1
- new net S_P: C16.1, C21.1, R5.2, R6.2, U13.14 (V+), U13.14 (V+), U13.14 (V+), U13.14 (V+), U20.14 (V+), U20.14 (V+)
Other:
- moved on the sheet: C115, C116, J1, J3, R75, R76, R77, R78, R79, U16

Commit message: begin PCB
Parts:
- removed C10, C11: 470nF, symbol C_Small
- removed C115: 100nF, symbol C_Small
- removed C75, C76: 2.2uF, symbol CP_Small
- removed C94: 220, symbol C_Small
- removed C95: 1uF, symbol CP_Small
- removed R105: 680, symbol R_Small
- removed R77: 100, symbol R_Small
- removed RN6: 4.7k, symbol R_Pack04
- removed U13: 4066, symbol 4066
- added C44, C45, C46: 100nF, UI:C_1206_0603, symbol C_Small
- added C48: 2.2uF, Capacitors_ThroughHole:CP_Radial_D4.0mm_P2.00mm, symbol CP_Small
- added C49: 1uF, Capacitors_ThroughHole:CP_Radial_D4.0mm_P2.00mm, symbol CP_Small
- added C50: 220, UI:C_1206_0603, symbol C_Small
- added K1: FRT5, Relays_ThroughHole:Relay_DPDT_FRT5, symbol FRT5
- added R19: 100, UI:R_1206_0603, symbol R_Small
- added R20: 680, UI:R_1206_0603, symbol R_Small
- C116: footprint (none) -> Capacitors_ThroughHole:CP_Radial_D5.0mm_P2.00mm
- C12, C13, C7, C8, C9: footprint (none) -> UI:C_1206_0603
- C14, C15, C17, C19: footprint (none) -> Capacitors_ThroughHole:CP_Radial_D4.0mm_P2.00mm
- D1: footprint (none) -> Diodes_SMD:D_MiniMELF_Handsoldering
- J1, J4: footprint (none) -> UI:audio_jack_3_5mm_PJ307
- J3: footprint LCSDR:audio_jack_3_5mm_PJ307 -> UI:audio_jack_3_5mm_PJ307
- R4, R75, R76, R78, R79: footprint (none) -> UI:R_1206_0603
- RN4, RN5, RN7: footprint (none) -> Resistors_SMD:R_Array_Convex_4x0603
- U20: footprint (none) -> Housings_SOIC:SOIC-14_3.9x8.7mm_Pitch1.27mm
Connections:
- net labels added: I2C_SCL, I2C_SDA
- net labels removed: I2C2_SCL, I2C2_SDA
- wire segments 184 -> 172
Other:
- moved on the sheet: C14, C15, J3, J4

Commit message: PCB update
Parts:
- removed C12, C13, C9: 470nF, UI:C_1206_0603, symbol C_Small
- removed C21: 100nF, symbol C_Small
- removed C48: 2.2uF, Capacitors_ThroughHole:CP_Radial_D4.0mm_P2.00mm, symbol CP_Small
- removed R78, R79: 100, UI:R_1206_0603, symbol R_Small
- removed RN4, RN5: 47, Resistors_SMD:R_Array_Convex_4x0603, symbol R_Pack04
- removed U20: 4066, Housings_SOIC:SOIC-14_3.9x8.7mm_Pitch1.27mm, symbol 4066
- added D4, D5: D_Small, Diodes_SMD:D_MiniMELF_Handsoldering, symbol D_Small
- added K2: FRT5, Relays_ThroughHole:Relay_DPDT_FRT5, symbol FRT5
- added Q1, Q2: Q_NPN_BEC, TO_SOT_Packages_SMD:SOT-23_Handsoldering, symbol Q_NPN_BEC
- C16: footprint (none) -> UI:C_1206_0603
- C5, C6: value 1nF -> 100nF; footprint (none) -> UI:C_1206_0603
- C8: value 470nF -> 100nF
- R5, R6: value 0* -> 2.2k; footprint (none) -> UI:R_1206_0603
Connections:
- net labels added: +12V, PTT_IN, TX1, TX2
- net labels removed: +9VA, I_IN_M1, I_IN_M2, LINE_OUT_LEFT_MCU, LINE_OUT_RIGHT_MCU, PTTIN, Q_IN_M1, Q_IN_M2, S_P
- wire segments 172 -> 157
Other:
- moved on the sheet: C14, C15, C16, J4, K1
