File: PCB/ST32_SDR/syntez.sch (KiCad schematic (older format))
At the start: 1 part, among them U12 STM32F103C8Tx

Commit message: add LCD resistors
Parts:
- removed U12: STM32F103C8Tx, Housings_QFP:LQFP-48_7x7mm_Pitch0.5mm, symbol STM32F103C8Tx
Changed lines of the file:
@@
 LIBS:contrib
 LIBS:LCSDR
+LIBS:Logic_74xx
+LIBS:Logic_CMOS_4000
 LIBS:4ms-ic
+LIBS:Connector
 LIBS:Display
+LIBS:TRXklopik
 LIBS:LCSDR-cache
 EELAYER 25 0
@@
 Comment4 ""
 $EndDescr
-$Comp
-L STM32F103C8Tx U12
-U 1 1 5DC33740
-P 5650 3350
-F 0 "U12" H 2850 5075 50  0000 L BNN
-F 1 "STM32F103C8Tx" H 8450 5075 50  0000 R BNN
-F 2 "Housings_QFP:LQFP-48_7x7mm_Pitch0.5mm" H 8450 5025 50  0001 R TNN
-F 3 "" H 5650 3350 50  0001 C CNN
-	1    5650 3350
-	1    0    0    -1
-$EndComp
 $EndSCHEMATC

Commit message: update schematics
Parts:
- added C1, C2, C3, C4: 100nF, symbol C_Small
- added R1, R2, R3: 100, symbol R_Small
- added RN3: 47, symbol R_Pack04
- added U1: SI5351A, MODULE, symbol SI5351A
- added Y2: Crystal, symbol Crystal
Connections:
- new net: C2.2, U1.10 (CLK0)
- new net: U1.2 (XA), Y2.2
- new net: U1.3 (XB), Y2.1
- new net: C4.2, U1.6 (CLK2)
- new net: C3.2, U1.9 (CLK1)
- new net +3V3: C1.1, U1.1 (VDD), U1.7 (VDDO)
- new net BAND0: RN3.1 (R1.1)
- new net BAND1: RN3.2 (R2.1)
- new net BAND2: RN3.3 (R3.1)
- new net BAND3: RN3.4 (R4.1)
- new net CLK0: C2.1, R1.1
- new net CLK1: C3.1, R2.1
- new net CLK2: C4.1, R3.1
- new net GND: C1.2, R1.2, R2.2, R3.2, U1.8 (GND)
- new net I2C_SCL: U1.4 (SCL)
- new net I2C_SDA: U1.5 (SDA)

Commit message: begin PCB
Parts:
- C1, C2, C3, C4: footprint (none) -> UI:C_1206_0603
- R1, R2, R3: footprint (none) -> UI:R_1206_0603
- RN3: footprint (none) -> Resistors_SMD:R_Array_Convex_4x0603
- U1: footprint MODULE -> Housings_SSOP:MSOP-10_3x3mm_Pitch0.5mm
- Y2: footprint (none) -> Crystals:Crystal_HC49-U_Vertical
Changed lines of the file:
@@
 LIBS:4ms-ic
 LIBS:Display
-LIBS:TRXklopik
-LIBS:stm32
-LIBS:switches
-LIBS:cmos4000
-LIBS:conn
+LIBS:Connector
+LIBS:Relay
 LIBS:LCSDR-cache
 EELAYER 25 0
@@
 F 0 "U1" H 4350 3010 50  0000 C CNN
 F 1 "SI5351A" H 4350 2925 50  0000 C CNN
-F 2 "MODULE" H 4350 2450 50  0001 C CNN
+F 2 "Housings_SSOP:MSOP-10_3x3mm_Pitch0.5mm" H 4350 2450 50  0001 C CNN
 F 3 "DOCUMENTATION" H 4370 2310 50  0001 C CNN
 	1    4350 2450
@@
 F 0 "Y2" H 3150 2350 50  0000 C CNN
 F 1 "Crystal" H 3150 2050 50  0000 C CNN
-F 2 "" H 3150 2200 50  0001 C CNN
+F 2 "Crystals:Crystal_HC49-U_Vertical" H 3150 2200 50  0001 C CNN
 F 3 "" H 3150 2200 50  0001 C CNN
 	1    3150 2200
@@
 F 0 "C1" V 3000 1700 50  0000 L CNN
 F 1 "100nF" V 3100 1700 50  0000 L CNN
-F 2 "" H 3250 1800 50  0001 C CNN
+F 2 "UI:C_1206_0603" H 3250 1800 50  0001 C CNN
 F 3 "" H 3250 1800 50  0001 C CNN
 	1    3250 1800
@@
 F 0 "C4" V 5600 2550 50  0000 L CNN
 F 1 "100nF" V 5700 2550 50  0000 L CNN
-F 2 "" H 5850 2650 50  0001 C CNN
+F 2 "UI:C_1206_0603" H 5850 2650 50  0001 C CNN
 F 3 "" H 5850 2650 50  0001 C CNN
 	1    5850 2650
@@
 F 0 "C3" V 5600 1750 50  0000 L CNN
 F 1 "100nF" V 5700 1750 50  0000 L CNN
-F 2 "" H 5850 1850 50  0001 C CNN
+F 2 "UI:C_1206_0603" H 5850 1850 50  0001 C CNN
 F 3 "" H 5850 1850 50  0001 C CNN
 	1    5850 1850
@@
 F 0 "C2" V 5600 1000 50  0000 L CNN
 F 1 "100nF" V 5700 1000 50  0000 L CNN
-F 2 "" H 5850 1100 50  0001 C CNN
+F 2 "UI:C_1206_0603" H 5850 1100 50  0001 C CNN
 F 3 "" H 5850 1100 50  0001 C CNN
 	1    5850 1100
@@
 F 0 "R1" H 6150 1350 50  0000 L CNN
 F 1 "100" H 6150 1250 50  0000 L CNN
-F 2 "" H 6100 1300 50  0001 C CNN
+F 2 "UI:R_1206_0603" H 6100 1300 50  0001 C CNN
 F 3 "" H 6100 1300 50  0001 C CNN
 	1    6100 1300
@@
 F 0 "R2" H 6150 2100 50  0000 L CNN
 F 1 "100" H 6150 2000 50  0000 L CNN
-F 2 "" H 6100 2050 50  0001 C CNN
+F 2 "UI:R_1206_0603" H 6100 2050 50  0001 C CNN
 F 3 "" H 6100 2050 50  0001 C CNN
 	1    6100 2050
@@
 F 0 "R3" H 6150 2900 50  0000 L CNN
 F 1 "100" H 6150 2800 50  0000 L CNN
-F 2 "" H 6100 2850 50  0001 C CNN
+F 2 "UI:R_1206_0603" H 6100 2850 50  0001 C CNN
 F 3 "" H 6100 2850 50  0001 C CNN
 	1    6100 2850
@@
 F 0 "RN3" V 3100 4600 50  0000 C CNN
 F 1 "47" V 3600 4600 50  0000 C CNN
-F 2 "" V 3675 4600 50  0001 C CNN
+F 2 "Resistors_SMD:R_Array_Convex_4x0603" V 3675 4600 50  0001 C CNN
 F 3 "" H 3400 4600 50  0001 C CNN
 	1    3400 4600

Commit message: PCB update
Parts:
- added R? (x2): 56, symbol R_Small
Connections:
- net BAND0: now also RN3.4 (R4.1); no longer RN3.1 (R1.1)
- net BAND1: now also RN3.3 (R3.1); no longer RN3.2 (R2.1)
- net BAND2: now also RN3.2 (R2.1); no longer RN3.3 (R3.1)
- net BAND3: now also RN3.1 (R1.1); no longer RN3.4 (R4.1)
- net I2C_SCL: now also R?.2
- net I2C_SDA: now also R?.2
- new net I2C_SCL_MCU: R?.1
- new net I2C_SDA_MCU: R?.1
Changed lines of the file:
@@
 	3550 2250 3700 2250
 Wire Wire Line
-	3550 1500 3550 2250
+	3550 1500 3550 1800
+Wire Wire Line
+	3550 1800 3550 2250
 $Comp
 L +3V3 #PWR01
@@
 Text GLabel 2550 2700 0    60   Input ~ 0
 I2C_SCL
-Text GLabel 2550 2900 0    60   Input ~ 0
+Text GLabel 2550 2900 0    60   BiDi ~ 0
 I2C_SDA
 Wire Wire Line
@@
 $EndComp
 Wire Wire Line
-	5950 1100 6500 1100
+	5950 1100 6100 1100
+Wire Wire Line
+	6100 1100 6500 1100
 Wire Wire Line
 	6100 1100 6100 1200
@@
 $EndComp
 Wire Wire Line
-	5950 1850 6500 1850
+	5950 1850 6100 1850
+Wire Wire Line
+	6100 1850 6500 1850
 Wire Wire Line
 	6100 1850 6100 1950
@@
 $EndComp
 Wire Wire Line
-	5950 2650 6500 2650
+	5950 2650 6100 2650
+Wire Wire Line
+	6100 2650 6500 2650
 Wire Wire Line
 	6100 2650 6100 2750
@@
 	0    1    1    0
 $EndComp
-Text GLabel 2850 4250 0    60   Input ~ 0
+Text GLabel 2750 4850 0    60   Input ~ 0
 BAND0
 Wire Wire Line
 	3000 4400 3200 4400
-Text GLabel 2850 4450 0    60   Input ~ 0
+Text GLabel 2750 4650 0    60   Input ~ 0
 BAND1
 Wire Wire Line
 	2900 4500 3200 4500
-Text GLabel 2850 4650 0    60   Input ~ 0
+Text GLabel 2750 4450 0    60   Input ~ 0
 BAND2
 Wire Wire Line
-	2850 4450 2900 4450
+	2750 4450 2900 4450
 Wire Wire Line
 	2900 4450 2900 4500
 Wire Wire Line
-	2850 4650 2900 4650
+	2750 4650 2900 4650
 Wire Wire Line
 	2900 4650 2900 4600
 Wire Wire Line
 	2900 4600 3200 4600
-Text GLabel 2850 4850 0    60   Input ~ 0
+Text GLabel 2750 4250 0    60   Input ~ 0
 BAND3
 Wire Wire Line
-	2850 4250 3000 4250
+	2750 4250 3000 4250
 Wire Wire Line
 	3000 4250 3000 4400
 Wire Wire Line
-	2850 4850 3000 4850
+	2750 4850 3000 4850
 Wire Wire Line
 	3000 4850 3000 4700
 Wire Wire Line
 	3000 4700 3200 4700
+Text GLabel 1300 1050 0    60   Input ~ 0
+I2C_SCL_MCU
+Text GLabel 1300 1300 0    60   BiDi ~ 0
+I2C_SDA_MCU
+$Comp
+L R_Small R?
+U 1 1 5DE23CAB
+P 1550 1050
+F 0 "R?" V 1750 1050 50  0000 L CNN
+F 1 "56" V 1650 1050 50  0000 L CNN
+F 2 "" H 1550 1050 50  0001 C CNN
+F 3 "" H 1550 1050 50  0001 C CNN
+	1    1550 1050
+	0    -1   -1   0
+$EndComp
+$Comp
+L R_Small R?
+U 1 1 5DE23D38
+P 1550 1300
+F 0 "R?" V 1450 1300 50  0000 L CNN
+F 1 "56" V 1350 1300 50  0000 L CNN
+F 2 "" H 1550 1300 50  0001 C CNN
+F 3 "" H 1550 1300 50  0001 C CNN
+	1    1550 1300
+	0    -1   -1   0
+$EndComp
+Text GLabel 1850 1050 2    60   Output ~ 0
+I2C_SCL
+Wire Wire Line
+	1450 1050 1300 1050
+Wire Wire Line
+	1650 1050 1850 1050
+Text GLabel 1850 1300 2    60   BiDi ~ 0
+I2C_SDA
+Wire Wire Line
+	1850 1300 1650 1300
+Wire Wire Line
+	1450 1300 1300 1300
 $EndSCHEMATC

Commit message: schematics update to privious commit
Parts:
- gave numbers to parts that had none: 2
Changed lines of the file:
@@
 	3550 2250 3700 2250
 Wire Wire Line
-	3550 1500 3550 1800
-Wire Wire Line
-	3550 1800 3550 2250
-$Comp
-L +3V3 #PWR01
+	3550 1500 3550 2250
+$Comp
+L +3V3 #PWR2
 U 1 1 5DDEDF62
 P 3550 1500
-F 0 "#PWR01" H 3550 1350 50  0001 C CNN
+F 0 "#PWR2" H 3550 1350 50  0001 C CNN
 F 1 "+3V3" H 3550 1640 50  0000 C CNN
 F 2 "" H 3550 1500 50  0001 C CNN
@@
 	3000 2900 2550 2900
 $Comp
-L GND #PWR02
+L GND #PWR1
 U 1 1 5DDEE4A0
 P 3150 1800
-F 0 "#PWR02" H 3150 1550 50  0001 C CNN
+F 0 "#PWR1" H 3150 1550 50  0001 C CNN
 F 1 "GND" H 3150 1650 50  0001 C CNN
 F 2 "" H 3150 1800 50  0001 C CNN
@@
 $EndComp
 $Comp
-L GND #PWR03
+L GND #PWR3
 U 1 1 5DDEE4E1
 P 5000 2450
-F 0 "#PWR03" H 5000 2200 50  0001 C CNN
+F 0 "#PWR3" H 5000 2200 50  0001 C CNN
 F 1 "GND" H 5000 2300 50  0001 C CNN
 F 2 "" H 5000 2450 50  0001 C CNN
@@
 $EndComp
 $Comp
-L +3V3 #PWR04
+L +3V3 #PWR4
 U 1 1 5DDEE519
 P 5000 2550
-F 0 "#PWR04" H 5000 2400 50  0001 C CNN
+F 0 "#PWR4" H 5000 2400 50  0001 C CNN
 F 1 "+3V3" V 5000 2800 50  0000 C CNN
 F 2 "" H 5000 2550 50  0001 C CNN
@@
 $EndComp
 Wire Wire Line
-	5950 1100 6100 1100
-Wire Wire Line
-	6100 1100 6500 1100
+	5950 1100 6500 1100
 Wire Wire Line
 	6100 1100 6100 1200
@@
 $EndComp
 Wire Wire Line
-	5950 1850 6100 1850
-Wire Wire Line
-	6100 1850 6500 1850
+	5950 1850 6500 1850
 Wire Wire Line
 	6100 1850 6100 1950
@@
 Connection ~ 6100 1100
 $Comp
-L GND #PWR05
+L GND #PWR5
 U 1 1 5DDEEBF2
 P 6100 1400
-F 0 "#PWR05" H 6100 1150 50  0001 C CNN
+F 0 "#PWR5" H 6100 1150 50  0001 C CNN
 F 1 "GND" H 6100 1250 50  0001 C CNN
 F 2 "" H 6100 1400 50  0001 C CNN
@@
 $EndComp
 $Comp
-L GND #PWR06
+L GND #PWR6
 U 1 1 5DDEEC35
 P 6100 2150
-F 0 "#PWR06" H 6100 1900 50  0001 C CNN
+F 0 "#PWR6" H 6100 1900 50  0001 C CNN
 F 1 "GND" H 6100 2000 50  0001 C CNN
 F 2 "" H 6100 2150 50  0001 C CNN
@@
 $EndComp
 Wire Wire Line
-	5950 2650 6100 2650
-Wire Wire Line
-	6100 2650 6500 2650
+	5950 2650 6500 2650
 Wire Wire Line
 	6100 2650 6100 2750
 $Comp
-L GND #PWR07
+L GND #PWR7
 U 1 1 5DDEECF7
 P 6100 2950
-F 0 "#PWR07" H 6100 2700 50  0001 C CNN
+F 0 "#PWR7" H 6100 2700 50  0001 C CNN
 F 1 "GND" H 6100 2800 50  0001 C CNN
 F 2 "" H 6100 2950 50  0001 C CNN
@@
 I2C_SDA_MCU
 $Comp
-L R_Small R?
+L R_Small R22
 U 1 1 5DE23CAB
 P 1550 1050
-F 0 "R?" V 1750 1050 50  0000 L CNN
+F 0 "R22" V 1750 1050 50  0000 L CNN
 F 1 "56" V 1650 1050 50  0000 L CNN
 F 2 "" H 1550 1050 50  0001 C CNN
@@
 $EndComp
 $Comp
-L R_Small R?
+L R_Small R23
 U 1 1 5DE23D38
 P 1550 1300
-F 0 "R?" V 1450 1300 50  0000 L CNN
+F 0 "R23" V 1450 1300 50  0000 L CNN
 F 1 "56" V 1350 1300 50  0000 L CNN
 F 2 "" H 1550 1300 50  0001 C CNN
